File: keyboard-layout/controller.kicad_pcb (KiCad board)
At the start: 2 copper layers, 90.2 x 41.9 mm, 23 parts, among them J1 USB_mini_micro_B, K1 KEYSW, K2 KEYSW, K3 KEYSW, K4 KEYSW, SW1 SW_PUSH, X1 XTAL_GND

Commit message: mx footprints
Parts:
- moved C6 21.3 mm to (144.5, 80.0), turned to 90 degrees
Connections:
- net /col0 renamed /Keyboard Matrix/col0
- net /col1 renamed /Keyboard Matrix/col1
- net /row0 renamed /Keyboard Matrix/row0
- net /row1 renamed /Keyboard Matrix/row1
Routing:
- net VCC: track 0.00 -> 111.4 mm
- net /Keyboard Matrix/col1: track 0.00 -> 83.5 mm, vias 0 -> 1
- net /Keyboard Matrix/col0: track 0.00 -> 63.0 mm, vias 0 -> 1
- net /Keyboard Matrix/row1: track 0.00 -> 60.3 mm, vias 0 -> 2
- net /Keyboard Matrix/row0: track 0.00 -> 52.0 mm, vias 0 -> 4
- net Net-(J1-Pad2): track 0.00 -> 49.5 mm, vias 0 -> 2
- net Net-(J1-Pad3): track 0.00 -> 46.4 mm, vias 0 -> 2
- net Net-(MCU1-Pad20): track 0.00 -> 34.2 mm, vias 0 -> 2
- net Net-(MCU1-Pad4): track 0.00 -> 16.2 mm
- net Net-(MCU1-Pad5): track 0.00 -> 13.8 mm
- net Net-(MCU1-Pad43): track 0.00 -> 12.7 mm
- net Net-(C7-Pad1): track 0.00 -> 12.4 mm
- net Net-(C2-Pad1): track 0.00 -> 12.0 mm
- net GND: track 0.00 -> 11.4 mm
- net Net-(C1-Pad1): track 0.00 -> 11.2 mm
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- removed copper zone on F.Cu, net GND
