File: keyboard-layout/Matrix.sch (KiCad schematic (older format))
At the start: 8 parts, among them K1 KEYSW, K2 KEYSW, K3 KEYSW, K4 KEYSW

Commit message: mx footprints
Connections:
- net col0: no longer K1.1, K3.1
- net col1: no longer K2.1, K4.1
- net row0: no longer D1.1 (K), D2.1 (K)
- net row1: no longer D3.1 (K), D4.1 (K)
Changed lines of the file:
@@
 $Descr A4 11693 8268
 encoding utf-8
-Sheet 2 2
+Sheet 2 3
 Title ""
 Date ""
@@
 $EndComp
 Wire Wire Line
-	2850 4050 2850 4150
-Wire Wire Line
-	2700 4150 3900 4150
-Wire Wire Line
-	3900 4150 3900 4050
-Wire Wire Line
-	3550 3650 3650 3650
-Wire Wire Line
-	3650 3450 3650 4450
-Wire Wire Line
-	3650 4450 3550 4450
-Wire Wire Line
-	4600 3650 4700 3650
-Wire Wire Line
-	4700 3450 4700 4450
-Wire Wire Line
-	4700 4450 4600 4450
-Wire Wire Line
 	3900 3750 3900 3650
 Wire Wire Line
 	3900 3650 4000 3650
-Wire Wire Line
-	2850 4850 2850 4950
-Wire Wire Line
-	2700 4950 3900 4950
-Wire Wire Line
-	3900 4950 3900 4850
 Wire Wire Line
 	3900 4550 3900 4450
@@
 Wire Wire Line
 	2850 4450 2950 4450
-Connection ~ 2850 4150
-Connection ~ 2850 4950
-Connection ~ 3650 3650
-Connection ~ 4700 3650
 Text HLabel 3650 3450 1    60   Input ~ 0
 col0

Commit message: Keyboard Matrix
Parts:
- removed D1, D2, D3, D4: D, keyboard_parts:D_SOD123_axial, symbol D
- removed K1, K2, K3, K4: KEYSW, mx1a:MX1A, symbol KEYSW
- added D? (x95): D, symbol D
- added K? (x95): KEYSW, symbol KEYSW
Connections:
- new net: D?.2 (A), K?.2 (x95)
