File: keyboard-layout/Matrix.sch (KiCad schematic (older format))
At the start: 190 parts, among them SW0 KEYSW, SW1 KEYSW, SW10 KEYSW, SW11 KEYSW, SW12 KEYSW, SW13 KEYSW, SW14 KEYSW, SW15 KEYSW, SW16 KEYSW, SW17 KEYSW, SW18 KEYSW, SW19 KEYSW, SW2 KEYSW, SW20 KEYSW, SW21 KEYSW, SW22 KEYSW, SW23 KEYSW, SW24 KEYSW, SW25 KEYSW, SW26 KEYSW, SW27 KEYSW, SW28 KEYSW, SW29 KEYSW, SW3 KEYSW, SW30 KEYSW, SW31 KEYSW, SW32 KEYSW, SW33 KEYSW, SW34 KEYSW, SW35 KEYSW, SW36 KEYSW, SW37 KEYSW, SW38 KEYSW, SW39 KEYSW, SW4 KEYSW, SW40 KEYSW, SW41 KEYSW, SW42 KEYSW, SW43 KEYSW, SW44 KEYSW, SW45 KEYSW, SW46 KEYSW, SW47 KEYSW, SW48 KEYSW, SW49 KEYSW, SW5 KEYSW, SW50 KEYSW, SW51 KEYSW, SW52 KEYSW, SW53 KEYSW, SW54 KEYSW, SW55 KEYSW, SW56 KEYSW, SW57 KEYSW, SW58 KEYSW, SW59 KEYSW, SW6 KEYSW, SW60 KEYSW, SW61 KEYSW, SW62 KEYSW, SW63 KEYSW, SW64 KEYSW, SW65 KEYSW, SW66 KEYSW, SW67 KEYSW, SW68 KEYSW, SW69 KEYSW, SW7 KEYSW, SW70 KEYSW, SW71 KEYSW, SW72 KEYSW, SW73 KEYSW, SW74 KEYSW, SW75 KEYSW, SW76 KEYSW, SW77 KEYSW, SW78 KEYSW, SW79 KEYSW, SW8 KEYSW, SW80 KEYSW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

Commit message: python scripting
Parts:
- removed D0, D1, D2, D3, D4, D5, D6, D7, D8: D, Diodes_SMD:D_SOD-123, symbol D
- removed SW0, SW1, SW2, SW3, SW4, SW5, SW6, SW7, SW8: KEYSW, symbol KEYSW
- renumbered D9 to D0, D10 to D1, D19 to D10, D20 to D11, D21 to D12, D22 to D13, D23 to D14, D24 to D15, D25 to D16, D26 to D17, D27 to D18, D28 to D19, D11 to D2, D29 to D20, D30 to D21, D31 to D22, D32 to D23, D33 to D24, D34 to D25, D35 to D26, D36 to D27, D37 to D28, D38 to D29, D12 to D3, D39 to D30, D40 to D31, D41 to D32, D42 to D33, D43 to D34, D44 to D35, D45 to D36, D46 to D37, D47 to D38, D48 to D39, D13 to D4, D49 to D40, D50 to D41, D51 to D42, D52 to D43, D53 to D44, D54 to D45, D55 to D46, D56 to D47, D57 to D48, D58 to D49, D14 to D5, D59 to D50, D60 to D51, D61 to D52, D62 to D53, D63 to D54, D64 to D55, D65 to D56, D66 to D57, D67 to D58, D68 to D59, D15 to D6, D69 to D60, D70 to D61, D71 to D62, D72 to D63, D73 to D64, D74 to D65, D75 to D66, D76 to D67, D77 to D68, D78 to D69, D16 to D7, D79 to D70, D80 to D71, D81 to D72, D82 to D73, D83 to D74, D84 to D75, D85 to D76, D86 to D77, D87 to D78, D88 to D79, D17 to D8, D89 to D80, D90 to D81, D91 to D82, D92 to D83, D93 to D84, D94 to D85, D18 to D9, SW9 to SW0, SW10 to SW1, SW19 to SW10, SW20 to SW11, SW21 to SW12, SW22 to SW13, SW23 to SW14, SW24 to SW15, SW25 to SW16, SW26 to SW17, SW27 to SW18, SW28 to SW19, SW11 to SW2, SW29 to SW20, SW30 to SW21, SW31 to SW22, SW32 to SW23, SW33 to SW24, SW34 to SW25, SW35 to SW26, SW36 to SW27, SW37 to SW28, SW38 to SW29, SW12 to SW3, SW39 to SW30, SW40 to SW31, SW41 to SW32, SW42 to SW33, SW43 to SW34, SW44 to SW35, SW45 to SW36, SW46 to SW37, SW47 to SW38, SW48 to SW39, SW13 to SW4, SW49 to SW40, SW50 to SW41, SW51 to SW42, SW52 to SW43, SW53 to SW44, SW54 to SW45, SW55 to SW46, SW56 to SW47, SW57 to SW48, SW58 to SW49, SW14 to SW5, SW59 to SW50, SW60 to SW51, SW61 to SW52, SW62 to SW53, SW63 to SW54, SW64 to SW55, SW65 to SW56, SW66 to SW57, SW67 to SW58, SW68 to SW59, SW15 to SW6, SW69 to SW60, SW70 to SW61, SW71 to SW62, SW72 to SW63, SW73 to SW64, SW74 to SW65, SW75 to SW66, SW76 to SW67, SW77 to SW68, SW78 to SW69, SW16 to SW7, SW79 to SW70, SW80 to SW71, SW81 to SW72, SW82 to SW73, SW83 to SW74, SW84 to SW75, SW85 to SW76, SW86 to SW77, SW87 to SW78, SW88 to SW79, SW17 to SW8, SW89 to SW80, SW90 to SW81, SW91 to SW82, SW92 to SW83, SW93 to SW84, SW94 to SW85, SW18 to SW9
Connections:
- net row5 is gone; now on net row4: D73.1 (K), D74.1 (K), D75.1 (K), D76.1 (K), D77.1 (K), D78.1 (K), D79.1 (K), D80.1 (K), D81.1 (K), D82.1 (K), D83.1 (K), D84.1 (K), D85.1 (K)
- net row0: now also D0.1 (K), D1.1 (K), D10.1 (K), D11.1 (K), D12.1 (K), D13.1 (K), D14.1 (K), D15.1 (K), D16.1 (K), D17.1 (K), D18.1 (K), D19.1 (K), D2.1 (K), D3.1 (K), D4.1 (K), D5.1 (K), D6.1 (K), D7.1 (K), D8.1 (K), D9.1 (K)
- net row1: now also D20.1 (K), D21.1 (K), D22.1 (K), D23.1 (K), D24.1 (K), D25.1 (K), D26.1 (K), D27.1 (K), D28.1 (K), D29.1 (K), D30.1 (K), D31.1 (K), D32.1 (K), D34.1 (K), D35.1 (K), D36.1 (K), D37.1 (K), D38.1 (K); no longer D0.1 (K), D1.1 (K), D10.1 (K), D11.1 (K), D12.1 (K), D13.1 (K), D14.1 (K), D15.1 (K), D16.1 (K), D17.1 (K), D18.1 (K), D19.1 (K), D2.1 (K), D3.1 (K), D4.1 (K), D5.1 (K), D6.1 (K), D7.1 (K), D8.1 (K), D9.1 (K)
- net row2: now also D33.1 (K), D39.1 (K), D40.1 (K), D41.1 (K), D42.1 (K), D43.1 (K), D44.1 (K), D45.1 (K), D46.1 (K), D47.1 (K), D48.1 (K), D49.1 (K), D50.1 (K), D51.1 (K), D52.1 (K), D53.1 (K), D54.1 (K), D55.1 (K); no longer D20.1 (K), D21.1 (K), D22.1 (K), D23.1 (K), D24.1 (K), D25.1 (K), D26.1 (K), D27.1 (K), D28.1 (K), D29.1 (K), D30.1 (K), D31.1 (K), D32.1 (K), D34.1 (K), D35.1 (K), D36.1 (K), D37.1 (K), D38.1 (K)
- net row3: now also D56.1 (K), D57.1 (K), D58.1 (K), D59.1 (K), D60.1 (K), D61.1 (K), D62.1 (K), D63.1 (K), D64.1 (K), D65.1 (K), D66.1 (K), D67.1 (K), D68.1 (K), D69.1 (K), D70.1 (K), D71.1 (K), D72.1 (K); no longer D33.1 (K), D39.1 (K), D40.1 (K), D41.1 (K), D42.1 (K), D43.1 (K), D44.1 (K), D45.1 (K), D46.1 (K), D47.1 (K), D48.1 (K), D49.1 (K), D50.1 (K), D51.1 (K), D52.1 (K), D53.1 (K), D54.1 (K), D55.1 (K)
- net row4: no longer D56.1 (K), D57.1 (K), D58.1 (K), D59.1 (K), D60.1 (K), D61.1 (K), D62.1 (K), D63.1 (K), D64.1 (K), D65.1 (K), D66.1 (K), D67.1 (K), D68.1 (K), D69.1 (K), D70.1 (K), D71.1 (K), D72.1 (K)

Commit message: pcb without leds finished
Changed lines of the file:
@@
 $Descr User 23622 11811
 encoding utf-8
-Sheet 2 3
+Sheet 3 3
 Title ""
 Date ""
@@
 	22000 3800 22000 3700
 Connection ~ 22000 3800
-Wire Wire Line
-	900  5600 22000 5600
 Connection ~ 9000 3300
 Connection ~ 2900 3300
@@
 	22000 5600 22000 5200
 Wire Wire Line
-	900  6500 21000 6500
-Wire Wire Line
 	22000 7400 22000 7300
 Wire Wire Line
@@
 Connection ~ 1100 6500
 Wire Wire Line
-	2100 6400 2100 6500
+	2100 6500 2100 6400
 Connection ~ 2100 6500
 Wire Wire Line
@@
 Text HLabel 900  5600 0    60   Input ~ 0
 row2
-Text HLabel 900  6500 0    60   Input ~ 0
-row3
 Text HLabel 900  7400 0    60   Input ~ 0
 row4
@@
 	8200 5500 8200 5600
 Connection ~ 8200 5600
+Wire Wire Line
+	900  5600 22000 5600
+Text HLabel 900  6500 0    60   Input ~ 0
+row3
+Wire Wire Line
+	900  6500 21000 6500
 $EndSCHEMATC
