File: keyboard-layout/keyboard-layout-pcb.kicad_pcb (KiCad board)
At the start: 2 copper layers, 95 parts, among them SW0 SW_MX, SW1 SW_MX, SW10 SW_MX, SW11 SW_MX, SW12 SW_MX, SW13 SW_MX, SW14 SW_MX, SW15 SW_MX, SW16 SW_MX, SW17 SW_MX, SW18 SW_MX, SW19 SW_MX, SW2 SW_MX, SW20 SW_MX, SW21 SW_MX, SW22 SW_MX, SW23 SW_MX, SW24 SW_MX, SW25 SW_MX, SW26 SW_MX, SW27 SW_MX, SW28 SW_MX, SW29 SW_MX, SW3 SW_MX, SW30 SW_MX, SW31 SW_MX, SW32 SW_MX, SW33 SW_MX, SW34 SW_MX, SW35 SW_MX, SW36 SW_MX, SW37 SW_MX, SW38 SW_MX, SW39 SW_MX, SW4 SW_MX, SW40 SW_MX, SW41 SW_MX, SW42 SW_MX, SW43 SW_MX, SW44 SW_MX, SW45 SW_MX, SW46 SW_MX, SW47 SW_MX, SW48 SW_MX, SW49 SW_MX, SW5 SW_MX, SW50 SW_MX, SW51 SW_MX, SW52 SW_MX, SW53 SW_MX, SW54 SW_MX, SW55 SW_MX, SW56 SW_MX, SW57 SW_MX, SW58 SW_MX, SW59 SW_MX, SW6 SW_MX, SW60 SW_MX, SW61 SW_MX, SW62 SW_MX, SW63 SW_MX, SW64 SW_MX, SW65 SW_MX, SW66 SW_MX, SW67 SW_MX, SW68 SW_MX, SW69 SW_MX, SW7 SW_MX, SW70 SW_MX, SW71 SW_MX, SW72 SW_MX, SW73 SW_MX, SW74 SW_MX, SW75 SW_MX, SW76 SW_MX, SW77 SW_MX, SW78 SW_MX, SW79 SW_MX, SW8 SW_MX, SW80 SW_MX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

Commit message: pcb progress
Parts:
- added C1, C2, C3: 0.1u, Capacitors_SMD:C_0805_HandSoldering, B.Cu at (0.00, 22.0)
- added C4: 4.7u, Capacitors_SMD:C_0805_HandSoldering, B.Cu at (0.00, 22.0)
- added C5: 1u, Capacitors_SMD:C_0805_HandSoldering, B.Cu at (0.00, 22.0)
- added C6, C7: 22p, Capacitors_SMD:C_0805_HandSoldering, B.Cu at (0.00, 22.0)
- added D0: D, keyboard_parts:D_SOD123W_hand, B.Cu at (137.0, 63.0)
- added D1: D, keyboard_parts:D_SOD123W_hand, B.Cu at (38.8, -3.50)
- added D10, D11, D12, D13, D14, D15, D16, D17, D18, D19, D20, D21, D22, D23, D24, D25, D26, D27, D28, D29, D3, D30, D31, D32, D33, D34, D35, D36, D37, D38, D39, D4, D40, D41, D42, D43, D44, D45, D46, D47, D48, D49, D5, D50, D51, D52, D53, D54, D55, D56, D57, D58, D59, D6, D60, D61, D62, D63, D64, D65, D66, D67, D68, D69, D7, D70, D71, D72, D73, D74, D75, D76, D77, D78, D79, D8, D80, D81, D82, D83, D84, D85, D86, D87, D88, D89, D9, D90, D91, D92, D93, D94: D, keyboard_parts:D_SOD123W_hand, B.Cu at (0.00, 22.0)
- added D2: D, keyboard_parts:D_SOD123W_hand, B.Cu at (-6.00, 25.0)
- added J1: USB_mini_micro_B, keyboard_parts:USB_miniB_hirose_5S8, B.Cu at (-11.2, 12.2)
- added MCU1: AT90USB1286, AT90USB1286-AU:QFP80P1600X1600X120-64N, B.Cu at (31.0, 28.0)
- added R1, R2: 22, Resistors_SMD:R_0805_HandSoldering, B.Cu at (0.00, 22.0)
- added R3, R4: 10k, Resistors_SMD:R_0805_HandSoldering, B.Cu at (0.00, 22.0)
- added SW_95: SW_PUSH, Buttons_Switches_SMD:SW_SPST_TL3342, B.Cu at (-14.5, 29.8)
- added X1: XTAL_GND, keyboard_parts:FA-238, B.Cu at (3.00, 32.2)
- SW0: value SW_MX -> Undo
- SW1: value SW_MX -> Redo
- SW10, SW11, SW12, SW13, SW14, SW15, SW16, SW17, SW18, SW19, SW2, SW20, SW21, SW22, SW23, SW24, SW25, SW26, SW27, SW28, SW29, SW3, SW30, SW31, SW32, SW33, SW34, SW35, SW36, SW37, SW38, SW39, SW4, SW40, SW41, SW42, SW43, SW44, SW45, SW46, SW47, SW48, SW49, SW5, SW50, SW51, SW52, SW53, SW54, SW55, SW56, SW57, SW58, SW59, SW6, SW60, SW61, SW62, SW63, SW64, SW65, SW66, SW67, SW68, SW69, SW7, SW70, SW71, SW72, SW73, SW74, SW75, SW76, SW77, SW78, SW79, SW8, SW80, SW81, SW82, SW83, SW84, SW85, SW86, SW87, SW88, SW89, SW9, SW90, SW91, SW92, SW93, SW94: value SW_MX -> KEYSW
Connections:
- SW0 pad 1: (no net) -> /Keyboard Matrix/col5
- SW0 pad 2: (no net) -> Net-(D0-Pad2)
- SW1 pad 1: (no net) -> /Keyboard Matrix/col6
- SW1 pad 2: (no net) -> Net-(D1-Pad2)
- SW10 pad 1: (no net) -> /Keyboard Matrix/col1
- SW10 pad 2: (no net) -> Net-(D10-Pad2)
- SW11 pad 1: (no net) -> /Keyboard Matrix/col2
- SW11 pad 2: (no net) -> Net-(D11-Pad2)
- SW12 pad 1: (no net) -> /Keyboard Matrix/col3
- SW12 pad 2: (no net) -> Net-(D12-Pad2)
- SW13 pad 1: (no net) -> /Keyboard Matrix/col4
- SW13 pad 2: (no net) -> Net-(D13-Pad2)
- SW14 pad 1: (no net) -> /Keyboard Matrix/col5
- SW14 pad 2: (no net) -> Net-(D14-Pad2)
- SW15 pad 1: (no net) -> /Keyboard Matrix/col6
- SW15 pad 2: (no net) -> Net-(D15-Pad2)
- SW16 pad 1: (no net) -> /Keyboard Matrix/col7
- SW16 pad 2: (no net) -> Net-(D16-Pad2)
- SW17 pad 1: (no net) -> /Keyboard Matrix/col8
- SW17 pad 2: (no net) -> Net-(D17-Pad2)
- SW18 pad 1: (no net) -> /Keyboard Matrix/col9
- SW18 pad 2: (no net) -> Net-(D18-Pad2)
- SW19 pad 1: (no net) -> /Keyboard Matrix/col10
- SW19 pad 2: (no net) -> Net-(D19-Pad2)
- SW2 pad 1: (no net) -> /Keyboard Matrix/col8
- SW2 pad 2: (no net) -> Net-(D2-Pad2)
- SW20 pad 1: (no net) -> /Keyboard Matrix/col11
- SW20 pad 2: (no net) -> Net-(D20-Pad2)
- SW21 pad 1: (no net) -> /Keyboard Matrix/col12
- SW21 pad 2: (no net) -> Net-(D21-Pad2)
- SW22 pad 1: (no net) -> /Keyboard Matrix/col14
- SW22 pad 2: (no net) -> Net-(D22-Pad2)
- SW23 pad 1: (no net) -> /Keyboard Matrix/col15
- SW23 pad 2: (no net) -> Net-(D23-Pad2)
- SW24 pad 1: (no net) -> /Keyboard Matrix/col16
- SW24 pad 2: (no net) -> Net-(D24-Pad2)
- SW25 pad 1: (no net) -> /Keyboard Matrix/col17
- SW25 pad 2: (no net) -> Net-(D25-Pad2)
- SW26 pad 1: (no net) -> /Keyboard Matrix/col18
- SW26 pad 2: (no net) -> Net-(D26-Pad2)
- SW27 pad 1: (no net) -> /Keyboard Matrix/col19
- SW27 pad 2: (no net) -> Net-(D27-Pad2)
- SW28 pad 1: (no net) -> /Keyboard Matrix/col20
- SW28 pad 2: (no net) -> Net-(D28-Pad2)
- SW29 pad 1: (no net) -> /Keyboard Matrix/col0
- SW29 pad 2: (no net) -> Net-(D29-Pad2)
- SW3 pad 1: (no net) -> /Keyboard Matrix/col9
- SW3 pad 2: (no net) -> Net-(D3-Pad2)
- SW30 pad 1: (no net) -> /Keyboard Matrix/col2
- SW30 pad 2: (no net) -> Net-(D30-Pad2)
- SW31 pad 1: (no net) -> /Keyboard Matrix/col3
- SW31 pad 2: (no net) -> Net-(D31-Pad2)
- SW32 pad 1: (no net) -> /Keyboard Matrix/col4
- SW32 pad 2: (no net) -> Net-(D32-Pad2)
- SW33 pad 1: (no net) -> /Keyboard Matrix/col5
- SW33 pad 2: (no net) -> Net-(D33-Pad2)
- SW34 pad 1: (no net) -> /Keyboard Matrix/col6
- SW34 pad 2: (no net) -> Net-(D34-Pad2)
- SW35 pad 1: (no net) -> /Keyboard Matrix/col7
- SW35 pad 2: (no net) -> Net-(D35-Pad2)
- SW36 pad 1: (no net) -> /Keyboard Matrix/col8
- SW36 pad 2: (no net) -> Net-(D36-Pad2)
- SW37 pad 1: (no net) -> /Keyboard Matrix/col9
- SW37 pad 2: (no net) -> Net-(D37-Pad2)
- SW38 pad 1: (no net) -> /Keyboard Matrix/col10
- SW38 pad 2: (no net) -> Net-(D38-Pad2)
- SW39 pad 1: (no net) -> /Keyboard Matrix/col11
- SW39 pad 2: (no net) -> Net-(D39-Pad2)
- SW4 pad 1: (no net) -> /Keyboard Matrix/col10
- SW4 pad 2: (no net) -> Net-(D4-Pad2)
- SW40 pad 1: (no net) -> /Keyboard Matrix/col12
- SW40 pad 2: (no net) -> Net-(D40-Pad2)
- SW41 pad 1: (no net) -> /Keyboard Matrix/col13
- SW41 pad 2: (no net) -> Net-(D41-Pad2)
- SW42 pad 1: (no net) -> /Keyboard Matrix/col14
- SW42 pad 2: (no net) -> Net-(D42-Pad2)
- SW43 pad 1: (no net) -> /Keyboard Matrix/col15
- SW43 pad 2: (no net) -> Net-(D43-Pad2)
- SW44 pad 1: (no net) -> /Keyboard Matrix/col16
- SW44 pad 2: (no net) -> Net-(D44-Pad2)
- SW45 pad 1: (no net) -> /Keyboard Matrix/col17
- SW45 pad 2: (no net) -> Net-(D45-Pad2)
- SW46 pad 1: (no net) -> /Keyboard Matrix/col18
- SW46 pad 2: (no net) -> Net-(D46-Pad2)
- SW47 pad 1: (no net) -> /Keyboard Matrix/col19
- SW47 pad 2: (no net) -> Net-(D47-Pad2)
- SW48 pad 1: (no net) -> /Keyboard Matrix/col20
- SW48 pad 2: (no net) -> Net-(D48-Pad2)
- SW49 pad 1: (no net) -> /Keyboard Matrix/col0
- SW49 pad 2: (no net) -> Net-(D49-Pad2)
- SW5 pad 1: (no net) -> /Keyboard Matrix/col11
- SW5 pad 2: (no net) -> Net-(D5-Pad2)
- SW50 pad 1: (no net) -> /Keyboard Matrix/col2
- SW50 pad 2: (no net) -> Net-(D50-Pad2)
- SW51 pad 1: (no net) -> /Keyboard Matrix/col3
- SW51 pad 2: (no net) -> Net-(D51-Pad2)
- SW52 pad 1: (no net) -> /Keyboard Matrix/col4
- SW52 pad 2: (no net) -> Net-(D52-Pad2)
- SW53 pad 1: (no net) -> /Keyboard Matrix/col5
- SW53 pad 2: (no net) -> Net-(D53-Pad2)
- SW54 pad 1: (no net) -> /Keyboard Matrix/col6
- SW54 pad 2: (no net) -> Net-(D54-Pad2)
- SW55 pad 1: (no net) -> /Keyboard Matrix/col7
- SW55 pad 2: (no net) -> Net-(D55-Pad2)
- SW56 pad 1: (no net) -> /Keyboard Matrix/col8
- SW56 pad 2: (no net) -> Net-(D56-Pad2)
- SW57 pad 1: (no net) -> /Keyboard Matrix/col9
- SW57 pad 2: (no net) -> Net-(D57-Pad2)
- SW58 pad 1: (no net) -> /Keyboard Matrix/col10
- SW58 pad 2: (no net) -> Net-(D58-Pad2)
- SW59 pad 1: (no net) -> /Keyboard Matrix/col11
- SW59 pad 2: (no net) -> Net-(D59-Pad2)
- SW6 pad 1: (no net) -> /Keyboard Matrix/col12
- SW6 pad 2: (no net) -> Net-(D6-Pad2)
- SW60 pad 1: (no net) -> /Keyboard Matrix/col12
- SW60 pad 2: (no net) -> Net-(D60-Pad2)
- SW61 pad 1: (no net) -> /Keyboard Matrix/col13
- SW61 pad 2: (no net) -> Net-(D61-Pad2)
- SW62 pad 1: (no net) -> /Keyboard Matrix/col17
- SW62 pad 2: (no net) -> Net-(D62-Pad2)
- SW63 pad 1: (no net) -> /Keyboard Matrix/col18
- SW63 pad 2: (no net) -> Net-(D63-Pad2)
- SW64 pad 1: (no net) -> /Keyboard Matrix/col19
- SW64 pad 2: (no net) -> Net-(D64-Pad2)
- SW65 pad 1: (no net) -> /Keyboard Matrix/col0
- SW65 pad 2: (no net) -> Net-(D65-Pad2)
- SW66 pad 1: (no net) -> /Keyboard Matrix/col1
- SW66 pad 2: (no net) -> Net-(D66-Pad2)
- SW67 pad 1: (no net) -> /Keyboard Matrix/col2
- SW67 pad 2: (no net) -> Net-(D67-Pad2)
- SW68 pad 1: (no net) -> /Keyboard Matrix/col3
- SW68 pad 2: (no net) -> Net-(D68-Pad2)
- SW69 pad 1: (no net) -> /Keyboard Matrix/col4
- SW69 pad 2: (no net) -> Net-(D69-Pad2)
- SW7 pad 1: (no net) -> /Keyboard Matrix/col13
- SW7 pad 2: (no net) -> Net-(D7-Pad2)
- SW70 pad 1: (no net) -> /Keyboard Matrix/col5
- SW70 pad 2: (no net) -> Net-(D70-Pad2)
- SW71 pad 1: (no net) -> /Keyboard Matrix/col6
- SW71 pad 2: (no net) -> Net-(D71-Pad2)
- SW72 pad 1: (no net) -> /Keyboard Matrix/col7
- SW72 pad 2: (no net) -> Net-(D72-Pad2)
- SW73 pad 1: (no net) -> /Keyboard Matrix/col8
- SW73 pad 2: (no net) -> Net-(D73-Pad2)
- SW74 pad 1: (no net) -> /Keyboard Matrix/col9
- SW74 pad 2: (no net) -> Net-(D74-Pad2)
- SW75 pad 1: (no net) -> /Keyboard Matrix/col10
- SW75 pad 2: (no net) -> Net-(D75-Pad2)
- SW76 pad 1: (no net) -> /Keyboard Matrix/col11
- SW76 pad 2: (no net) -> Net-(D76-Pad2)
- SW77 pad 1: (no net) -> /Keyboard Matrix/col13
- SW77 pad 2: (no net) -> Net-(D77-Pad2)
- SW78 pad 1: (no net) -> /Keyboard Matrix/col15
- SW78 pad 2: (no net) -> Net-(D78-Pad2)
- SW79 pad 1: (no net) -> /Keyboard Matrix/col17
- SW79 pad 2: (no net) -> Net-(D79-Pad2)
- SW8 pad 1: (no net) -> /Keyboard Matrix/col14
- SW8 pad 2: (no net) -> Net-(D8-Pad2)
- SW80 pad 1: (no net) -> /Keyboard Matrix/col18
- SW80 pad 2: (no net) -> Net-(D80-Pad2)
- SW81 pad 1: (no net) -> /Keyboard Matrix/col19
- SW81 pad 2: (no net) -> Net-(D81-Pad2)
- SW82 pad 1: (no net) -> /Keyboard Matrix/col20
- SW82 pad 2: (no net) -> Net-(D82-Pad2)
- SW83 pad 1: (no net) -> /Keyboard Matrix/col0
- SW83 pad 2: (no net) -> Net-(D83-Pad2)
- SW84 pad 1: (no net) -> /Keyboard Matrix/col1
- SW84 pad 2: (no net) -> Net-(D84-Pad2)
- SW85 pad 1: (no net) -> /Keyboard Matrix/col3
- SW85 pad 2: (no net) -> Net-(D85-Pad2)
- SW86 pad 1: (no net) -> /Keyboard Matrix/col6
- SW86 pad 2: (no net) -> Net-(D86-Pad2)
- SW87 pad 1: (no net) -> /Keyboard Matrix/col10
- SW87 pad 2: (no net) -> Net-(D87-Pad2)
- SW88 pad 1: (no net) -> /Keyboard Matrix/col11
- SW88 pad 2: (no net) -> Net-(D88-Pad2)
- SW89 pad 1: (no net) -> /Keyboard Matrix/col13
- SW89 pad 2: (no net) -> Net-(D89-Pad2)
- SW9 pad 1: (no net) -> /Keyboard Matrix/col0
- SW9 pad 2: (no net) -> Net-(D9-Pad2)
- SW90 pad 1: (no net) -> /Keyboard Matrix/col14
- SW90 pad 2: (no net) -> Net-(D90-Pad2)
- SW91 pad 1: (no net) -> /Keyboard Matrix/col15
- SW91 pad 2: (no net) -> Net-(D91-Pad2)
- SW92 pad 1: (no net) -> /Keyboard Matrix/col16
- SW92 pad 2: (no net) -> Net-(D92-Pad2)
- SW93 pad 1: (no net) -> /Keyboard Matrix/col17
- SW93 pad 2: (no net) -> Net-(D93-Pad2)
- SW94 pad 1: (no net) -> /Keyboard Matrix/col19
- SW94 pad 2: (no net) -> Net-(D94-Pad2)

Commit message: python scripting
Parts:
- removed D0, D1, D2, D3, D4, D5, D6, D7, D8: D, keyboard_parts:D_SOD123W_hand
- removed SW0: Undo, Button_Switch_Keyboard:SW_Cherry_MX1A_1.00u_PCB
- removed SW1: Redo, Button_Switch_Keyboard:SW_Cherry_MX1A_1.00u_PCB
- removed SW2, SW3, SW4, SW5, SW6, SW7, SW8: KEYSW, Button_Switch_Keyboard:SW_Cherry_MX1A_1.00u_PCB
- moved D82 458.9 mm to (439.4, 154.4), turned to 180 degrees
- moved D48 449.4 mm to (439.4, 116.4), turned to 180 degrees
- moved D28 444.3 mm to (439.4, 87.9), turned to 180 degrees
- moved D81 438.0 mm to (420.4, 144.9), turned to 180 degrees
- moved D64 433.0 mm to (420.4, 125.9), turned to 180 degrees
- moved D47 428.9 mm to (420.4, 106.9), turned to 180 degrees
- moved D27 425.5 mm to (420.4, 87.9), turned to 180 degrees
- moved D80 419.8 mm to (401.4, 144.9), turned to 180 degrees
- moved D93 416.8 mm to (391.9, 163.9), turned to 180 degrees
- moved D63 414.6 mm to (401.4, 125.9), turned to 180 degrees
- moved D46 410.3 mm to (401.4, 106.9), turned to 180 degrees
- moved D26 406.7 mm to (401.4, 87.9), turned to 180 degrees
- moved D79 401.6 mm to (382.4, 144.9), turned to 180 degrees
- moved D62 396.2 mm to (382.4, 125.9), turned to 180 degrees
- moved D45 391.7 mm to (382.4, 106.9), turned to 180 degrees
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Connections:
- D10 pad 1: /Keyboard Matrix/row1 -> /Keyboard Matrix/row0
- D11 pad 1: /Keyboard Matrix/row1 -> /Keyboard Matrix/row0
- D12 pad 1: /Keyboard Matrix/row1 -> /Keyboard Matrix/row0
- D13 pad 1: /Keyboard Matrix/row1 -> /Keyboard Matrix/row0
- D14 pad 1: /Keyboard Matrix/row1 -> /Keyboard Matrix/row0
- D15 pad 1: /Keyboard Matrix/row1 -> /Keyboard Matrix/row0
- D16 pad 1: /Keyboard Matrix/row1 -> /Keyboard Matrix/row0
- D17 pad 1: /Keyboard Matrix/row1 -> /Keyboard Matrix/row0
- D18 pad 1: /Keyboard Matrix/row1 -> /Keyboard Matrix/row0
- D19 pad 1: /Keyboard Matrix/row1 -> /Keyboard Matrix/row0
- D20 pad 1: /Keyboard Matrix/row1 -> /Keyboard Matrix/row0
- D21 pad 1: /Keyboard Matrix/row1 -> /Keyboard Matrix/row0
- D22 pad 1: /Keyboard Matrix/row1 -> /Keyboard Matrix/row0
- D23 pad 1: /Keyboard Matrix/row1 -> /Keyboard Matrix/row0
- D24 pad 1: /Keyboard Matrix/row1 -> /Keyboard Matrix/row0
- D25 pad 1: /Keyboard Matrix/row1 -> /Keyboard Matrix/row0
- D26 pad 1: /Keyboard Matrix/row1 -> /Keyboard Matrix/row0
- D27 pad 1: /Keyboard Matrix/row1 -> /Keyboard Matrix/row0
- D28 pad 1: /Keyboard Matrix/row1 -> /Keyboard Matrix/row0
- D29 pad 1: /Keyboard Matrix/row2 -> /Keyboard Matrix/row1
- D30 pad 1: /Keyboard Matrix/row2 -> /Keyboard Matrix/row1
- D31 pad 1: /Keyboard Matrix/row2 -> /Keyboard Matrix/row1
- D32 pad 1: /Keyboard Matrix/row2 -> /Keyboard Matrix/row1
- D33 pad 1: /Keyboard Matrix/row2 -> /Keyboard Matrix/row1
- D34 pad 1: /Keyboard Matrix/row2 -> /Keyboard Matrix/row1
- D35 pad 1: /Keyboard Matrix/row2 -> /Keyboard Matrix/row1
- D36 pad 1: /Keyboard Matrix/row2 -> /Keyboard Matrix/row1
- D37 pad 1: /Keyboard Matrix/row2 -> /Keyboard Matrix/row1
- D38 pad 1: /Keyboard Matrix/row2 -> /Keyboard Matrix/row1
- D39 pad 1: /Keyboard Matrix/row2 -> /Keyboard Matrix/row1
- D40 pad 1: /Keyboard Matrix/row2 -> /Keyboard Matrix/row1
- D41 pad 1: /Keyboard Matrix/row2 -> /Keyboard Matrix/row1
- D43 pad 1: /Keyboard Matrix/row2 -> /Keyboard Matrix/row1
- D44 pad 1: /Keyboard Matrix/row2 -> /Keyboard Matrix/row1
- D45 pad 1: /Keyboard Matrix/row2 -> /Keyboard Matrix/row1
- D46 pad 1: /Keyboard Matrix/row2 -> /Keyboard Matrix/row1
- D47 pad 1: /Keyboard Matrix/row2 -> /Keyboard Matrix/row1
- D65 pad 1: /Keyboard Matrix/row4 -> /Keyboard Matrix/row2
- D66 pad 1: /Keyboard Matrix/row4 -> /Keyboard Matrix/row2
- D67 pad 1: /Keyboard Matrix/row4 -> /Keyboard Matrix/row2
- D68 pad 1: /Keyboard Matrix/row4 -> /Keyboard Matrix/row2
- D69 pad 1: /Keyboard Matrix/row4 -> /Keyboard Matrix/row2
- D70 pad 1: /Keyboard Matrix/row4 -> /Keyboard Matrix/row2
- D71 pad 1: /Keyboard Matrix/row4 -> /Keyboard Matrix/row2
- D72 pad 1: /Keyboard Matrix/row4 -> /Keyboard Matrix/row2
- D73 pad 1: /Keyboard Matrix/row4 -> /Keyboard Matrix/row2
- D74 pad 1: /Keyboard Matrix/row4 -> /Keyboard Matrix/row2
- D75 pad 1: /Keyboard Matrix/row4 -> /Keyboard Matrix/row2
- D76 pad 1: /Keyboard Matrix/row4 -> /Keyboard Matrix/row2
- D77 pad 1: /Keyboard Matrix/row4 -> /Keyboard Matrix/row2
- D78 pad 1: /Keyboard Matrix/row4 -> /Keyboard Matrix/row2
- D79 pad 1: /Keyboard Matrix/row4 -> /Keyboard Matrix/row2
- D80 pad 1: /Keyboard Matrix/row4 -> /Keyboard Matrix/row2
- D81 pad 1: /Keyboard Matrix/row4 -> /Keyboard Matrix/row2
- D82 pad 1: /Keyboard Matrix/row5 -> /Keyboard Matrix/row4
- D83 pad 1: /Keyboard Matrix/row5 -> /Keyboard Matrix/row4
- D84 pad 1: /Keyboard Matrix/row5 -> /Keyboard Matrix/row4
- D85 pad 1: /Keyboard Matrix/row5 -> /Keyboard Matrix/row4
- D86 pad 1: /Keyboard Matrix/row5 -> /Keyboard Matrix/row4
- D87 pad 1: /Keyboard Matrix/row5 -> /Keyboard Matrix/row4
- D88 pad 1: /Keyboard Matrix/row5 -> /Keyboard Matrix/row4
- D89 pad 1: /Keyboard Matrix/row5 -> /Keyboard Matrix/row4
- D9 pad 1: /Keyboard Matrix/row1 -> /Keyboard Matrix/row0
- D90 pad 1: /Keyboard Matrix/row5 -> /Keyboard Matrix/row4
- D91 pad 1: /Keyboard Matrix/row5 -> /Keyboard Matrix/row4
- D92 pad 1: /Keyboard Matrix/row5 -> /Keyboard Matrix/row4
- D93 pad 1: /Keyboard Matrix/row5 -> /Keyboard Matrix/row4
- D94 pad 1: /Keyboard Matrix/row5 -> /Keyboard Matrix/row4
- MCU1 pad 56: /Keyboard Matrix/row5 -> Net-(MCU1-Pad56)

Commit message: Fresh
Parts:
- removed the SW13 at (125.9, 83.1)
- removed the SW39 at (249.4, 102.1)
- removed the SW77 at (299.2, 140.1)
- removed SW87, SW88, SW89: KEYSW, Button_Switch_Keyboard:SW_Cherry_MX1A_1.25u_PCB
- removed SW90, SW91, SW92, SW94: KEYSW, Button_Switch_Keyboard:SW_Cherry_MX1A_1.00u_PCB
- removed SW93: KEYSW, Button_Switch_Keyboard:SW_Cherry_MX1A_2.00u_PCB
- added SW0: Esc, Button_Switch_Keyboard:SW_Cherry_MX1A_1.00u_PCB, F.Cu at (49.9, 83.1)
- added SW1: 1, Button_Switch_Keyboard:SW_Cherry_MX1A_1.00u_PCB, F.Cu at (68.9, 83.1)
- added SW2: 2, Button_Switch_Keyboard:SW_Cherry_MX1A_1.00u_PCB, F.Cu at (87.9, 83.1)
- added SW22: W, Button_Switch_Keyboard:SW_Cherry_MX1A_1.00u_PCB, F.Cu at (97.4, 102.1)
- added SW3: 3, Button_Switch_Keyboard:SW_Cherry_MX1A_1.00u_PCB, F.Cu at (106.9, 83.1)
- added SW4: 4, Button_Switch_Keyboard:SW_Cherry_MX1A_1.00u_PCB, F.Cu at (125.9, 83.1)
- added SW48: K, Button_Switch_Keyboard:SW_Cherry_MX1A_1.00u_PCB, F.Cu at (216.1, 121.1)
- added SW5: 5, Button_Switch_Keyboard:SW_Cherry_MX1A_1.00u_PCB, F.Cu at (144.9, 83.1)
- added SW6: 6, Button_Switch_Keyboard:SW_Cherry_MX1A_1.00u_PCB, F.Cu at (163.9, 83.1)
- added SW7: 7, Button_Switch_Keyboard:SW_Cherry_MX1A_1.00u_PCB, F.Cu at (182.9, 83.1)
- added SW8: 8, Button_Switch_Keyboard:SW_Cherry_MX1A_1.00u_PCB, F.Cu at (201.9, 83.1)
- SW10: value KEYSW -> 0
- SW11, SW19: value KEYSW -> -
- SW12: value KEYSW -> =
- SW13: renamed from SW22; value KEYSW -> BkSp
- SW14: value KEYSW -> Light
- SW15: value KEYSW -> PgUp
- SW16: value KEYSW -> %
- SW17, SW67: value KEYSW -> /
- SW18: value KEYSW -> *
- SW20: value KEYSW -> Tab; footprint Button_Switch_Keyboard:SW_Cherry_MX1A_1.00u_PCB -> Button_Switch_Keyboard:SW_Cherry_MX1A_1.50u_PCB
- SW21: value KEYSW -> Q
- SW23: value KEYSW -> E
- SW24: value KEYSW -> R
- SW25: value KEYSW -> T
- SW26: value KEYSW -> Y
- SW27: value KEYSW -> U
- SW28: value KEYSW -> I
- SW29: value KEYSW -> O; footprint Button_Switch_Keyboard:SW_Cherry_MX1A_1.50u_PCB -> Button_Switch_Keyboard:SW_Cherry_MX1A_1.00u_PCB
- SW30: value KEYSW -> P
- SW31: value KEYSW -> [
- SW32: value KEYSW -> ]
- SW33: value KEYSW -> Return; footprint Button_Switch_Keyboard:SW_Cherry_MX1A_1.00u_PCB -> Button_Switch_Keyboard:SW_Cherry_MX1A_ISOEnter_PCB
- SW34: value KEYSW -> Del
- SW35: value KEYSW -> PgDw
- SW36: value KEYSW -> 7
- SW37: value KEYSW -> 8
- SW38, SW9: value KEYSW -> 9
- SW39: renamed from SW48; value KEYSW -> +
- SW40: value KEYSW -> Caps; footprint Button_Switch_Keyboard:SW_Cherry_MX1A_1.00u_PCB -> Button_Switch_Keyboard:SW_Cherry_MX1A_1.75u_PCB
- SW41: value KEYSW -> A
- SW42: value KEYSW -> S; footprint Button_Switch_Keyboard:SW_Cherry_MX1A_ISOEnter_PCB -> Button_Switch_Keyboard:SW_Cherry_MX1A_1.00u_PCB
- SW43: value KEYSW -> D
- SW44: value KEYSW -> F
- SW45: value KEYSW -> G
- SW46: value KEYSW -> H
- SW47: value KEYSW -> J
- SW49: value KEYSW -> L; footprint Button_Switch_Keyboard:SW_Cherry_MX1A_1.75u_PCB -> Button_Switch_Keyboard:SW_Cherry_MX1A_1.00u_PCB
- SW50: value KEYSW -> ;
- SW51: value KEYSW -> '
- SW52: value KEYSW -> \
- SW53: value KEYSW -> 4
- SW54: value KEYSW -> 5
- SW55: value KEYSW -> 6
- SW56: value KEYSW -> Lshft; footprint Button_Switch_Keyboard:SW_Cherry_MX1A_1.00u_PCB -> Button_Switch_Keyboard:SW_Cherry_MX1A_1.25u_PCB
- SW57: value KEYSW -> `
- SW58: value KEYSW -> Z
- SW59: value KEYSW -> X
- SW60: value KEYSW -> C
- SW61: value KEYSW -> V
- SW62: value KEYSW -> B
- SW63: value KEYSW -> N
- SW64: value KEYSW -> M
- SW65: value KEYSW -> ,; footprint Button_Switch_Keyboard:SW_Cherry_MX1A_1.25u_PCB -> Button_Switch_Keyboard:SW_Cherry_MX1A_1.00u_PCB
- SW66: value KEYSW -> .
- SW68: value KEYSW -> Rshft; footprint Button_Switch_Keyboard:SW_Cherry_MX1A_1.00u_PCB -> Button_Switch_Keyboard:SW_Cherry_MX1A_2.75u_PCB
- SW69: value KEYSW -> Up
- SW70: value KEYSW -> 1
- SW71: value KEYSW -> 2
- SW72: value KEYSW -> 3
- SW73: value KEYSW -> Ret; footprint Button_Switch_Keyboard:SW_Cherry_MX1A_1.00u_PCB -> Button_Switch_Keyboard:SW_Cherry_MX1A_2.00u_Vertical_PCB
- SW74: value KEYSW -> Ctrl; footprint Button_Switch_Keyboard:SW_Cherry_MX1A_1.00u_PCB -> Button_Switch_Keyboard:SW_Cherry_MX1A_1.25u_PCB
- SW75, SW79: value KEYSW -> Alt; footprint Button_Switch_Keyboard:SW_Cherry_MX1A_1.00u_PCB -> Button_Switch_Keyboard:SW_Cherry_MX1A_1.25u_PCB
- SW76, SW78: value KEYSW -> Cmd; footprint Button_Switch_Keyboard:SW_Cherry_MX1A_1.00u_PCB -> Button_Switch_Keyboard:SW_Cherry_MX1A_1.25u_PCB
- SW77: renamed from SW86; value KEYSW -> Space
- SW80: value KEYSW -> Fn; footprint Button_Switch_Keyboard:SW_Cherry_MX1A_1.00u_PCB -> Button_Switch_Keyboard:SW_Cherry_MX1A_1.25u_PCB
- SW81: value KEYSW -> Left
- SW82: value KEYSW -> Down; footprint Button_Switch_Keyboard:SW_Cherry_MX1A_2.00u_Vertical_PCB -> Button_Switch_Keyboard:SW_Cherry_MX1A_1.00u_PCB
- SW83: value KEYSW -> Right; footprint Button_Switch_Keyboard:SW_Cherry_MX1A_1.25u_PCB -> Button_Switch_Keyboard:SW_Cherry_MX1A_1.00u_PCB
- SW84: value KEYSW -> 0; footprint Button_Switch_Keyboard:SW_Cherry_MX1A_1.25u_PCB -> Button_Switch_Keyboard:SW_Cherry_MX1A_2.00u_PCB
- SW85: footprint Button_Switch_Keyboard:SW_Cherry_MX1A_1.25u_PCB -> Button_Switch_Keyboard:SW_Cherry_MX1A_1.00u_PCB
- moved D85 443.7 mm to (420.4, 163.9), turned to 180 degrees
- moved SW85 320.6 mm to (420.4, 159.1)
- moved SW84 315.9 mm to (391.9, 159.1)
- moved SW83 306.4 mm to (358.6, 159.1)
- moved SW53 242.2 mm to (382.4, 121.1)
- moved SW54 242.2 mm to (401.4, 121.1)
- moved SW55 242.2 mm to (420.4, 121.1)
- moved SW73 232.9 mm to (439.4, 149.6)
- moved SW70 232.8 mm to (382.4, 140.1)
- moved SW71 232.8 mm to (401.4, 140.1)
- moved SW72 232.8 mm to (420.4, 140.1)
- moved SW25 228.8 mm to (154.4, 102.1)
- moved SW26 228.8 mm to (173.4, 102.1)
- moved SW27 228.8 mm to (192.4, 102.1)
- moved SW28 228.8 mm to (211.4, 102.1)
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- renumbered D9 to D0, D10 to D1, D19 to D10, D20 to D11, D21 to D12, D22 to D13, D23 to D14, D24 to D15, D25 to D16, D26 to D17, D27 to D18, D28 to D19, D11 to D2, D29 to D20, D30 to D21, D31 to D22, D32 to D23, D33 to D24, D34 to D25, D35 to D26, D36 to D27, D37 to D28, D38 to D29, D12 to D3, D39 to D30, D40 to D31, D41 to D32, D42 to D33, D43 to D34, D44 to D35, D45 to D36, D46 to D37, D47 to D38, D48 to D39, D13 to D4, D49 to D40, D50 to D41, D51 to D42, D52 to D43, D53 to D44, D54 to D45, D55 to D46, D56 to D47, D57 to D48, D58 to D49, D14 to D5, D59 to D50, D60 to D51, D61 to D52, D62 to D53, D63 to D54, D64 to D55, D65 to D56, D66 to D57, D67 to D58, D68 to D59, D15 to D6, D69 to D60, D70 to D61, D71 to D62, D72 to D63, D73 to D64, D74 to D65, D75 to D66, D76 to D67, D77 to D68, D78 to D69, D16 to D7, D79 to D70, D80 to D71, D81 to D72, D82 to D73, D83 to D74, D84 to D75, D85 to D76, D86 to D77, D87 to D78, D88 to D79, D17 to D8, D89 to D80, D90 to D81, D91 to D82, D92 to D83, D93 to D84, D94 to D85, D18 to D9
Connections:
- D0 pad 2: Net-(D9-Pad2) -> Net-(D0-Pad2)
- D1 pad 2: Net-(D10-Pad2) -> Net-(D1-Pad2)
- D10 pad 2: Net-(D19-Pad2) -> Net-(D10-Pad2)
- D11 pad 2: Net-(D20-Pad2) -> Net-(D11-Pad2)
- D12 pad 2: Net-(D21-Pad2) -> Net-(D12-Pad2)
- D14 pad 2: Net-(D23-Pad2) -> Net-(D14-Pad2)
- D15 pad 2: Net-(D24-Pad2) -> Net-(D15-Pad2)
- D16 pad 2: Net-(D25-Pad2) -> Net-(D16-Pad2)
- D17 pad 2: Net-(D26-Pad2) -> Net-(D17-Pad2)
- D18 pad 2: Net-(D27-Pad2) -> Net-(D18-Pad2)
- D19 pad 2: Net-(D28-Pad2) -> Net-(D19-Pad2)
- D2 pad 2: Net-(D11-Pad2) -> Net-(D2-Pad2)
- D20 pad 2: Net-(D29-Pad2) -> Net-(D20-Pad2)
- D21 pad 2: Net-(D30-Pad2) -> Net-(D21-Pad2)
- D22 pad 2: Net-(D31-Pad2) -> Net-(D22-Pad2)
- D23 pad 2: Net-(D32-Pad2) -> Net-(D23-Pad2)
- D24 pad 2: Net-(D33-Pad2) -> Net-(D24-Pad2)
- D25 pad 2: Net-(D34-Pad2) -> Net-(D25-Pad2)
- D26 pad 2: Net-(D35-Pad2) -> Net-(D26-Pad2)
- D27 pad 2: Net-(D36-Pad2) -> Net-(D27-Pad2)
- D28 pad 2: Net-(D37-Pad2) -> Net-(D28-Pad2)
- D29 pad 2: Net-(D38-Pad2) -> Net-(D29-Pad2)
- D3 pad 2: Net-(D12-Pad2) -> Net-(D3-Pad2)
- D30 pad 2: Net-(D39-Pad2) (its old number) -> Net-(D30-Pad2)
- D31 pad 2: Net-(D40-Pad2) -> Net-(D31-Pad2)
- D32 pad 2: Net-(D41-Pad2) -> Net-(D32-Pad2)
- D33 pad 2: Net-(D42-Pad2) -> Net-(D33-Pad2)
- D34 pad 2: Net-(D43-Pad2) -> Net-(D34-Pad2)
- D35 pad 2: Net-(D44-Pad2) -> Net-(D35-Pad2)
- D36 pad 2: Net-(D45-Pad2) -> Net-(D36-Pad2)
- D37 pad 2: Net-(D46-Pad2) -> Net-(D37-Pad2)
- D38 pad 2: Net-(D47-Pad2) -> Net-(D38-Pad2)
- D40 pad 2: Net-(D49-Pad2) -> Net-(D40-Pad2)
- D41 pad 2: Net-(D50-Pad2) -> Net-(D41-Pad2)
- D42 pad 2: Net-(D51-Pad2) -> Net-(D42-Pad2)
- D43 pad 2: Net-(D52-Pad2) -> Net-(D43-Pad2)
- D44 pad 2: Net-(D53-Pad2) -> Net-(D44-Pad2)
- D45 pad 2: Net-(D54-Pad2) -> Net-(D45-Pad2)
- D46 pad 2: Net-(D55-Pad2) -> Net-(D46-Pad2)
- D47 pad 2: Net-(D56-Pad2) -> Net-(D47-Pad2)
- D48 pad 2: Net-(D57-Pad2) -> Net-(D48-Pad2)
- D49 pad 2: Net-(D58-Pad2) -> Net-(D49-Pad2)
- D5 pad 2: Net-(D14-Pad2) -> Net-(D5-Pad2)
- D50 pad 2: Net-(D59-Pad2) -> Net-(D50-Pad2)
- D51 pad 2: Net-(D60-Pad2) -> Net-(D51-Pad2)
- D52 pad 2: Net-(D61-Pad2) -> Net-(D52-Pad2)
- D53 pad 2: Net-(D62-Pad2) -> Net-(D53-Pad2)
- D54 pad 2: Net-(D63-Pad2) -> Net-(D54-Pad2)
- D55 pad 2: Net-(D64-Pad2) -> Net-(D55-Pad2)
- D56 pad 2: Net-(D65-Pad2) -> Net-(D56-Pad2)
- D57 pad 2: Net-(D66-Pad2) -> Net-(D57-Pad2)
- D58 pad 2: Net-(D67-Pad2) -> Net-(D58-Pad2)
- D59 pad 2: Net-(D68-Pad2) -> Net-(D59-Pad2)
- D6 pad 2: Net-(D15-Pad2) -> Net-(D6-Pad2)
- D60 pad 2: Net-(D69-Pad2) -> Net-(D60-Pad2)
- D61 pad 2: Net-(D70-Pad2) -> Net-(D61-Pad2)
- D62 pad 2: Net-(D71-Pad2) -> Net-(D62-Pad2)
- D63 pad 2: Net-(D72-Pad2) -> Net-(D63-Pad2)
- D64 pad 2: Net-(D73-Pad2) -> Net-(D64-Pad2)
- D65 pad 2: Net-(D74-Pad2) -> Net-(D65-Pad2)
- D66 pad 2: Net-(D75-Pad2) -> Net-(D66-Pad2)
- D67 pad 2: Net-(D76-Pad2) -> Net-(D67-Pad2)
- D68 pad 2: Net-(D77-Pad2) (its old number) -> Net-(D68-Pad2)
- D69 pad 2: Net-(D78-Pad2) -> Net-(D69-Pad2)
- D7 pad 2: Net-(D16-Pad2) -> Net-(D7-Pad2)
- D70 pad 2: Net-(D79-Pad2) -> Net-(D70-Pad2)
- D71 pad 2: Net-(D80-Pad2) -> Net-(D71-Pad2)
- D72 pad 2: Net-(D81-Pad2) -> Net-(D72-Pad2)
- D73 pad 2: Net-(D82-Pad2) -> Net-(D73-Pad2)
- D74 pad 2: Net-(D83-Pad2) -> Net-(D74-Pad2)
- D75 pad 2: Net-(D84-Pad2) -> Net-(D75-Pad2)
- D76 pad 2: Net-(D85-Pad2) -> Net-(D76-Pad2)
- D78 pad 2: Net-(D87-Pad2) -> Net-(D78-Pad2)
- D79 pad 2: Net-(D88-Pad2) -> Net-(D79-Pad2)
- D8 pad 2: Net-(D17-Pad2) -> Net-(D8-Pad2)
- D80 pad 2: Net-(D89-Pad2) -> Net-(D80-Pad2)
- D81 pad 2: Net-(D90-Pad2) -> Net-(D81-Pad2)
- D82 pad 2: Net-(D91-Pad2) -> Net-(D82-Pad2)
- D83 pad 2: Net-(D92-Pad2) -> Net-(D83-Pad2)
- D84 pad 2: Net-(D93-Pad2) -> Net-(D84-Pad2)
- D85 pad 2: Net-(D94-Pad2) -> Net-(D85-Pad2)
- D9 pad 2: Net-(D18-Pad2) -> Net-(D9-Pad2)
- SW10 pad 1: /Keyboard Matrix/col1 -> /Keyboard Matrix/col10
- SW11 pad 1: /Keyboard Matrix/col2 -> /Keyboard Matrix/col11
- SW12 pad 1: /Keyboard Matrix/col3 -> /Keyboard Matrix/col12
- SW14 pad 1: /Keyboard Matrix/col5 -> /Keyboard Matrix/col15
- SW15 pad 1: /Keyboard Matrix/col6 -> /Keyboard Matrix/col16
- SW16 pad 1: /Keyboard Matrix/col7 -> /Keyboard Matrix/col17
- SW17 pad 1: /Keyboard Matrix/col8 -> /Keyboard Matrix/col18
- SW18 pad 1: /Keyboard Matrix/col9 -> /Keyboard Matrix/col19
- SW19 pad 1: /Keyboard Matrix/col10 -> /Keyboard Matrix/col20
- SW20 pad 1: /Keyboard Matrix/col11 -> /Keyboard Matrix/col0
- SW21 pad 1: /Keyboard Matrix/col12 -> /Keyboard Matrix/col2
- SW23 pad 1: /Keyboard Matrix/col15 -> /Keyboard Matrix/col4
- SW24 pad 1: /Keyboard Matrix/col16 -> /Keyboard Matrix/col5
- SW25 pad 1: /Keyboard Matrix/col17 -> /Keyboard Matrix/col6
- SW26 pad 1: /Keyboard Matrix/col18 -> /Keyboard Matrix/col7
- SW27 pad 1: /Keyboard Matrix/col19 -> /Keyboard Matrix/col8
- SW28 pad 1: /Keyboard Matrix/col20 -> /Keyboard Matrix/col9
- SW29 pad 1: /Keyboard Matrix/col0 -> /Keyboard Matrix/col10
- SW30 pad 1: /Keyboard Matrix/col2 -> /Keyboard Matrix/col11
- SW31 pad 1: /Keyboard Matrix/col3 -> /Keyboard Matrix/col12
- SW32 pad 1: /Keyboard Matrix/col4 -> /Keyboard Matrix/col13
- SW33 pad 1: /Keyboard Matrix/col5 -> /Keyboard Matrix/col14
- SW34 pad 1: /Keyboard Matrix/col6 -> /Keyboard Matrix/col15
- SW35 pad 1: /Keyboard Matrix/col7 -> /Keyboard Matrix/col16
- SW36 pad 1: /Keyboard Matrix/col8 -> /Keyboard Matrix/col17
- SW37 pad 1: /Keyboard Matrix/col9 -> /Keyboard Matrix/col18
- SW38 pad 1: /Keyboard Matrix/col10 -> /Keyboard Matrix/col19
- SW40 pad 1: /Keyboard Matrix/col12 -> /Keyboard Matrix/col0
- SW41 pad 1: /Keyboard Matrix/col13 -> /Keyboard Matrix/col2
- SW42 pad 1: /Keyboard Matrix/col14 -> /Keyboard Matrix/col3
- SW43 pad 1: /Keyboard Matrix/col15 -> /Keyboard Matrix/col4
- SW44 pad 1: /Keyboard Matrix/col16 -> /Keyboard Matrix/col5
- SW45 pad 1: /Keyboard Matrix/col17 -> /Keyboard Matrix/col6
- SW46 pad 1: /Keyboard Matrix/col18 -> /Keyboard Matrix/col7
- SW47 pad 1: /Keyboard Matrix/col19 -> /Keyboard Matrix/col8
- SW49 pad 1: /Keyboard Matrix/col0 -> /Keyboard Matrix/col10
- SW50 pad 1: /Keyboard Matrix/col2 -> /Keyboard Matrix/col11
- SW51 pad 1: /Keyboard Matrix/col3 -> /Keyboard Matrix/col12
- SW52 pad 1: /Keyboard Matrix/col4 -> /Keyboard Matrix/col13
- SW53 pad 1: /Keyboard Matrix/col5 -> /Keyboard Matrix/col17
- SW54 pad 1: /Keyboard Matrix/col6 -> /Keyboard Matrix/col18
- SW55 pad 1: /Keyboard Matrix/col7 -> /Keyboard Matrix/col19
- SW56 pad 1: /Keyboard Matrix/col8 -> /Keyboard Matrix/col0
- SW57 pad 1: /Keyboard Matrix/col9 -> /Keyboard Matrix/col1
- SW58 pad 1: /Keyboard Matrix/col10 -> /Keyboard Matrix/col2
- SW59 pad 1: /Keyboard Matrix/col11 -> /Keyboard Matrix/col3
- SW60 pad 1: /Keyboard Matrix/col12 -> /Keyboard Matrix/col4
- SW61 pad 1: /Keyboard Matrix/col13 -> /Keyboard Matrix/col5
- SW62 pad 1: /Keyboard Matrix/col17 -> /Keyboard Matrix/col6
- SW63 pad 1: /Keyboard Matrix/col18 -> /Keyboard Matrix/col7
- SW64 pad 1: /Keyboard Matrix/col19 -> /Keyboard Matrix/col8
- SW65 pad 1: /Keyboard Matrix/col0 -> /Keyboard Matrix/col9
- SW66 pad 1: /Keyboard Matrix/col1 -> /Keyboard Matrix/col10
- SW67 pad 1: /Keyboard Matrix/col2 -> /Keyboard Matrix/col11
- SW68 pad 1: /Keyboard Matrix/col3 -> /Keyboard Matrix/col13
- SW69 pad 1: /Keyboard Matrix/col4 -> /Keyboard Matrix/col15
- SW70 pad 1: /Keyboard Matrix/col5 -> /Keyboard Matrix/col17
- SW71 pad 1: /Keyboard Matrix/col6 -> /Keyboard Matrix/col18
- SW72 pad 1: /Keyboard Matrix/col7 -> /Keyboard Matrix/col19
- SW73 pad 1: /Keyboard Matrix/col8 -> /Keyboard Matrix/col20
- SW74 pad 1: /Keyboard Matrix/col9 -> /Keyboard Matrix/col0
- SW75 pad 1: /Keyboard Matrix/col10 -> /Keyboard Matrix/col1
- SW76 pad 1: /Keyboard Matrix/col11 -> /Keyboard Matrix/col3
- SW78 pad 1: /Keyboard Matrix/col15 -> /Keyboard Matrix/col10
- SW79 pad 1: /Keyboard Matrix/col17 -> /Keyboard Matrix/col11
- SW80 pad 1: /Keyboard Matrix/col18 -> /Keyboard Matrix/col13
- SW81 pad 1: /Keyboard Matrix/col19 -> /Keyboard Matrix/col14
- SW82 pad 1: /Keyboard Matrix/col20 -> /Keyboard Matrix/col15
- SW83 pad 1: /Keyboard Matrix/col0 -> /Keyboard Matrix/col16
- SW84 pad 1: /Keyboard Matrix/col1 -> /Keyboard Matrix/col17
- SW85 pad 1: /Keyboard Matrix/col3 -> /Keyboard Matrix/col19
- SW9 pad 1: /Keyboard Matrix/col0 -> /Keyboard Matrix/col9

Commit message: cutting edge
Parts:
- moved C3 393.5 mm to (345.6, 210.2), turned to 180 degrees
- moved R3 387.6 mm to (351.5, 185.2), turned to 90 degrees
- moved C2 385.2 mm to (336.1, 210.2)
- moved C6 382.0 mm to (345.6, 184.9), turned to 270 degrees
- moved C4 375.5 mm to (328.9, 203.1), turned to 90 degrees
- moved C7 373.0 mm to (335.6, 184.9), turned to 90 degrees
- moved C5 372.7 mm to (328.9, 197.1), turned to 270 degrees
- moved X1 370.5 mm to (340.6, 184.9), turned to 225 degrees
- moved C1 364.4 mm to (330.1, 186.4), turned to 180 degrees
- moved MCU1 353.4 mm to (340.9, 197.8)
- moved R4 22.3 mm to (-10.7, 41.6), turned to 90 degrees
- moved R1 14.4 mm to (-14.2, 20.2)
- moved SW_95 12.4 mm to (-18.1, 41.6)
- moved R2 8.51 mm to (-8.31, 20.2)
Routing:
- added copper zone on B.Cu, net GND
- added copper zone on F.Cu, net GND
Other:
- board outline added: 413.2 x 99.8 mm
