File: keyboard-layout/keyboard-layout-pcb.kicad_pcb (KiCad board)
At the start: 2 copper layers, 413.2 x 99.8 mm, 187 parts, among them J1 USB_mini_micro_B, SW0 Esc, SW1 1, SW10 0, SW11 -, SW12 =, SW13 BkSp, SW14 Light, SW15 PgUp, SW16 %, SW17 /, SW18 *, SW19 -, SW2 2, SW20 Tab, SW21 Q, SW22 W, SW23 E, SW24 R, SW25 T, SW26 Y, SW27 U, SW28 I, SW29 O, SW3 3, SW30 P, SW31 [, SW32 ], SW33 Return, SW34 Del, SW35 PgDw, SW36 7, SW37 8, SW38 9, SW39 +, SW4 4, SW40 Caps, SW41 A, SW42 S, SW43 D, SW44 F, SW45 G, SW46 H, SW47 J, SW48 K, SW49 L, SW5 5, SW50 ;, SW51 ', SW52 \, SW53 4, SW54 5, SW55 6, SW56 Lshft, SW57 `, SW58 Z, SW59 X, SW6 6, SW60 C, SW61 V, SW62 B, SW63 N, SW64 M, SW65 ,, SW66 ., SW67 /, SW68 Rshft, SW69 Up, SW7 7, SW70 1, SW71 2, SW72 3, SW73 Ret, SW74 Ctrl, SW75 Alt, SW76 Cmd, SW77 Space, SW78 Cmd, SW79 Alt, SW8 8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

Commit message: pcb without leds finished
Parts:
- SW0: value Esc -> KEYSW; footprint Button_Switch_Keyboard:SW_Cherry_MX1A_1.00u_PCB -> Button_Switch_Keyboard:SW_Cherry_MX1A_1.00u_Plate
- SW1, SW70: value 1 -> KEYSW; footprint Button_Switch_Keyboard:SW_Cherry_MX1A_1.00u_PCB -> Button_Switch_Keyboard:SW_Cherry_MX1A_1.00u_Plate
- SW10: value 0 -> KEYSW; footprint Button_Switch_Keyboard:SW_Cherry_MX1A_1.00u_PCB -> Button_Switch_Keyboard:SW_Cherry_MX1A_1.00u_Plate
- SW11, SW19: value - -> KEYSW; footprint Button_Switch_Keyboard:SW_Cherry_MX1A_1.00u_PCB -> Button_Switch_Keyboard:SW_Cherry_MX1A_1.00u_Plate
- SW12: value = -> KEYSW; footprint Button_Switch_Keyboard:SW_Cherry_MX1A_1.00u_PCB -> Button_Switch_Keyboard:SW_Cherry_MX1A_1.00u_Plate
- SW13: value BkSp -> KEYSW; footprint Button_Switch_Keyboard:SW_Cherry_MX1A_2.00u_PCB -> Button_Switch_Keyboard:SW_Cherry_MX1A_2.00u_Plate
- SW14: value Light -> KEYSW; footprint Button_Switch_Keyboard:SW_Cherry_MX1A_1.00u_PCB -> Button_Switch_Keyboard:SW_Cherry_MX1A_1.00u_Plate
- SW15: value PgUp -> KEYSW; footprint Button_Switch_Keyboard:SW_Cherry_MX1A_1.00u_PCB -> Button_Switch_Keyboard:SW_Cherry_MX1A_1.00u_Plate
- SW16: value % -> KEYSW; footprint Button_Switch_Keyboard:SW_Cherry_MX1A_1.00u_PCB -> Button_Switch_Keyboard:SW_Cherry_MX1A_1.00u_Plate
- SW17, SW67: value / -> KEYSW; footprint Button_Switch_Keyboard:SW_Cherry_MX1A_1.00u_PCB -> Button_Switch_Keyboard:SW_Cherry_MX1A_1.00u_Plate
- SW18: value * -> KEYSW; footprint Button_Switch_Keyboard:SW_Cherry_MX1A_1.00u_PCB -> Button_Switch_Keyboard:SW_Cherry_MX1A_1.00u_Plate
- SW2, SW71: value 2 -> KEYSW; footprint Button_Switch_Keyboard:SW_Cherry_MX1A_1.00u_PCB -> Button_Switch_Keyboard:SW_Cherry_MX1A_1.00u_Plate
- SW20: value Tab -> KEYSW; footprint Button_Switch_Keyboard:SW_Cherry_MX1A_1.50u_PCB -> Button_Switch_Keyboard:SW_Cherry_MX1A_1.50u_Plate
- SW21: value Q -> KEYSW; footprint Button_Switch_Keyboard:SW_Cherry_MX1A_1.00u_PCB -> Button_Switch_Keyboard:SW_Cherry_MX1A_1.00u_Plate
- SW22: value W -> KEYSW; footprint Button_Switch_Keyboard:SW_Cherry_MX1A_1.00u_PCB -> Button_Switch_Keyboard:SW_Cherry_MX1A_1.00u_Plate
- SW23: value E -> KEYSW; footprint Button_Switch_Keyboard:SW_Cherry_MX1A_1.00u_PCB -> Button_Switch_Keyboard:SW_Cherry_MX1A_1.00u_Plate
- SW24: value R -> KEYSW; footprint Button_Switch_Keyboard:SW_Cherry_MX1A_1.00u_PCB -> Button_Switch_Keyboard:SW_Cherry_MX1A_1.00u_Plate
- SW25: value T -> KEYSW; footprint Button_Switch_Keyboard:SW_Cherry_MX1A_1.00u_PCB -> Button_Switch_Keyboard:SW_Cherry_MX1A_1.00u_Plate
- SW26: value Y -> KEYSW; footprint Button_Switch_Keyboard:SW_Cherry_MX1A_1.00u_PCB -> Button_Switch_Keyboard:SW_Cherry_MX1A_1.00u_Plate
- SW27: value U -> KEYSW; footprint Button_Switch_Keyboard:SW_Cherry_MX1A_1.00u_PCB -> Button_Switch_Keyboard:SW_Cherry_MX1A_1.00u_Plate
- SW28: value I -> KEYSW; footprint Button_Switch_Keyboard:SW_Cherry_MX1A_1.00u_PCB -> Button_Switch_Keyboard:SW_Cherry_MX1A_1.00u_Plate
- SW29: value O -> KEYSW; footprint Button_Switch_Keyboard:SW_Cherry_MX1A_1.00u_PCB -> Button_Switch_Keyboard:SW_Cherry_MX1A_1.00u_Plate
- SW3, SW72: value 3 -> KEYSW; footprint Button_Switch_Keyboard:SW_Cherry_MX1A_1.00u_PCB -> Button_Switch_Keyboard:SW_Cherry_MX1A_1.00u_Plate
- SW30: value P -> KEYSW; footprint Button_Switch_Keyboard:SW_Cherry_MX1A_1.00u_PCB -> Button_Switch_Keyboard:SW_Cherry_MX1A_1.00u_Plate
- SW31: value [ -> KEYSW; footprint Button_Switch_Keyboard:SW_Cherry_MX1A_1.00u_PCB -> Button_Switch_Keyboard:SW_Cherry_MX1A_1.00u_Plate
- SW32: value ] -> KEYSW; footprint Button_Switch_Keyboard:SW_Cherry_MX1A_1.00u_PCB -> Button_Switch_Keyboard:SW_Cherry_MX1A_1.00u_Plate
- SW33: value Return -> KEYSW; footprint Button_Switch_Keyboard:SW_Cherry_MX1A_ISOEnter_PCB -> Button_Switch_Keyboard:SW_Cherry_MX1A_ISOEnter_Plate
- SW34: value Del -> KEYSW; footprint Button_Switch_Keyboard:SW_Cherry_MX1A_1.00u_PCB -> Button_Switch_Keyboard:SW_Cherry_MX1A_1.00u_Plate
- SW35: value PgDw -> KEYSW; footprint Button_Switch_Keyboard:SW_Cherry_MX1A_1.00u_PCB -> Button_Switch_Keyboard:SW_Cherry_MX1A_1.00u_Plate
- SW36, SW7: value 7 -> KEYSW; footprint Button_Switch_Keyboard:SW_Cherry_MX1A_1.00u_PCB -> Button_Switch_Keyboard:SW_Cherry_MX1A_1.00u_Plate
- SW37, SW8: value 8 -> KEYSW; footprint Button_Switch_Keyboard:SW_Cherry_MX1A_1.00u_PCB -> Button_Switch_Keyboard:SW_Cherry_MX1A_1.00u_Plate
- SW38, SW9: value 9 -> KEYSW; footprint Button_Switch_Keyboard:SW_Cherry_MX1A_1.00u_PCB -> Button_Switch_Keyboard:SW_Cherry_MX1A_1.00u_Plate
- SW39: value + -> KEYSW; footprint Button_Switch_Keyboard:SW_Cherry_MX1A_2.00u_Vertical_PCB -> Button_Switch_Keyboard:SW_Cherry_MX1A_2.00u_Vertical_Plate
- SW4, SW53: value 4 -> KEYSW; footprint Button_Switch_Keyboard:SW_Cherry_MX1A_1.00u_PCB -> Button_Switch_Keyboard:SW_Cherry_MX1A_1.00u_Plate
- SW40: value Caps -> KEYSW; footprint Button_Switch_Keyboard:SW_Cherry_MX1A_1.75u_PCB -> Button_Switch_Keyboard:SW_Cherry_MX1A_1.75u_Plate
- SW41: value A -> KEYSW; footprint Button_Switch_Keyboard:SW_Cherry_MX1A_1.00u_PCB -> Button_Switch_Keyboard:SW_Cherry_MX1A_1.00u_Plate
- SW42: value S -> KEYSW; footprint Button_Switch_Keyboard:SW_Cherry_MX1A_1.00u_PCB -> Button_Switch_Keyboard:SW_Cherry_MX1A_1.00u_Plate
- SW43: value D -> KEYSW; footprint Button_Switch_Keyboard:SW_Cherry_MX1A_1.00u_PCB -> Button_Switch_Keyboard:SW_Cherry_MX1A_1.00u_Plate
- SW44: value F -> KEYSW; footprint Button_Switch_Keyboard:SW_Cherry_MX1A_1.00u_PCB -> Button_Switch_Keyboard:SW_Cherry_MX1A_1.00u_Plate
- SW45: value G -> KEYSW; footprint Button_Switch_Keyboard:SW_Cherry_MX1A_1.00u_PCB -> Button_Switch_Keyboard:SW_Cherry_MX1A_1.00u_Plate
- SW46: value H -> KEYSW; footprint Button_Switch_Keyboard:SW_Cherry_MX1A_1.00u_PCB -> Button_Switch_Keyboard:SW_Cherry_MX1A_1.00u_Plate
- SW47: value J -> KEYSW; footprint Button_Switch_Keyboard:SW_Cherry_MX1A_1.00u_PCB -> Button_Switch_Keyboard:SW_Cherry_MX1A_1.00u_Plate
- SW48: value K -> KEYSW; footprint Button_Switch_Keyboard:SW_Cherry_MX1A_1.00u_PCB -> Button_Switch_Keyboard:SW_Cherry_MX1A_1.00u_Plate
- SW49: value L -> KEYSW; footprint Button_Switch_Keyboard:SW_Cherry_MX1A_1.00u_PCB -> Button_Switch_Keyboard:SW_Cherry_MX1A_1.00u_Plate
- SW5, SW54: value 5 -> KEYSW; footprint Button_Switch_Keyboard:SW_Cherry_MX1A_1.00u_PCB -> Button_Switch_Keyboard:SW_Cherry_MX1A_1.00u_Plate
- SW50: value ; -> KEYSW; footprint Button_Switch_Keyboard:SW_Cherry_MX1A_1.00u_PCB -> Button_Switch_Keyboard:SW_Cherry_MX1A_1.00u_Plate
- SW51: value ' -> KEYSW; footprint Button_Switch_Keyboard:SW_Cherry_MX1A_1.00u_PCB -> Button_Switch_Keyboard:SW_Cherry_MX1A_1.00u_Plate
- SW52: value \ -> KEYSW; footprint Button_Switch_Keyboard:SW_Cherry_MX1A_1.00u_PCB -> Button_Switch_Keyboard:SW_Cherry_MX1A_1.00u_Plate
- SW55, SW6: value 6 -> KEYSW; footprint Button_Switch_Keyboard:SW_Cherry_MX1A_1.00u_PCB -> Button_Switch_Keyboard:SW_Cherry_MX1A_1.00u_Plate
- SW56: value Lshft -> KEYSW; footprint Button_Switch_Keyboard:SW_Cherry_MX1A_1.25u_PCB -> Button_Switch_Keyboard:SW_Cherry_MX1A_1.25u_Plate
- SW57: value ` -> KEYSW; footprint Button_Switch_Keyboard:SW_Cherry_MX1A_1.00u_PCB -> Button_Switch_Keyboard:SW_Cherry_MX1A_1.00u_Plate
- SW58: value Z -> KEYSW; footprint Button_Switch_Keyboard:SW_Cherry_MX1A_1.00u_PCB -> Button_Switch_Keyboard:SW_Cherry_MX1A_1.00u_Plate
- SW59: value X -> KEYSW; footprint Button_Switch_Keyboard:SW_Cherry_MX1A_1.00u_PCB -> Button_Switch_Keyboard:SW_Cherry_MX1A_1.00u_Plate
- SW60: value C -> KEYSW; footprint Button_Switch_Keyboard:SW_Cherry_MX1A_1.00u_PCB -> Button_Switch_Keyboard:SW_Cherry_MX1A_1.00u_Plate
- SW61: value V -> KEYSW; footprint Button_Switch_Keyboard:SW_Cherry_MX1A_1.00u_PCB -> Button_Switch_Keyboard:SW_Cherry_MX1A_1.00u_Plate
- SW62: value B -> KEYSW; footprint Button_Switch_Keyboard:SW_Cherry_MX1A_1.00u_PCB -> Button_Switch_Keyboard:SW_Cherry_MX1A_1.00u_Plate
- SW63: value N -> KEYSW; footprint Button_Switch_Keyboard:SW_Cherry_MX1A_1.00u_PCB -> Button_Switch_Keyboard:SW_Cherry_MX1A_1.00u_Plate
- SW64: value M -> KEYSW; footprint Button_Switch_Keyboard:SW_Cherry_MX1A_1.00u_PCB -> Button_Switch_Keyboard:SW_Cherry_MX1A_1.00u_Plate
- SW65: value , -> KEYSW; footprint Button_Switch_Keyboard:SW_Cherry_MX1A_1.00u_PCB -> Button_Switch_Keyboard:SW_Cherry_MX1A_1.00u_Plate
- SW66: value . -> KEYSW; footprint Button_Switch_Keyboard:SW_Cherry_MX1A_1.00u_PCB -> Button_Switch_Keyboard:SW_Cherry_MX1A_1.00u_Plate
- SW68: value Rshft -> KEYSW; footprint Button_Switch_Keyboard:SW_Cherry_MX1A_2.75u_PCB -> Button_Switch_Keyboard:SW_Cherry_MX1A_2.75u_Plate
- SW69: value Up -> KEYSW; footprint Button_Switch_Keyboard:SW_Cherry_MX1A_1.00u_PCB -> Button_Switch_Keyboard:SW_Cherry_MX1A_1.00u_Plate
- SW73: value Ret -> KEYSW; footprint Button_Switch_Keyboard:SW_Cherry_MX1A_2.00u_Vertical_PCB -> Button_Switch_Keyboard:SW_Cherry_MX1A_2.00u_Vertical_Plate
- SW74: value Ctrl -> KEYSW; footprint Button_Switch_Keyboard:SW_Cherry_MX1A_1.25u_PCB -> Button_Switch_Keyboard:SW_Cherry_MX1A_1.25u_Plate
- SW75, SW79: value Alt -> KEYSW; footprint Button_Switch_Keyboard:SW_Cherry_MX1A_1.25u_PCB -> Button_Switch_Keyboard:SW_Cherry_MX1A_1.25u_Plate
- SW76, SW78: value Cmd -> KEYSW; footprint Button_Switch_Keyboard:SW_Cherry_MX1A_1.25u_PCB -> Button_Switch_Keyboard:SW_Cherry_MX1A_1.25u_Plate
- SW77: value Space -> KEYSW; footprint Button_Switch_Keyboard:SW_Cherry_MX1A_6.25u_PCB -> Button_Switch_Keyboard:SW_Cherry_MX1A_6.25u_Plate
- SW80: value Fn -> KEYSW; footprint Button_Switch_Keyboard:SW_Cherry_MX1A_1.25u_PCB -> Button_Switch_Keyboard:SW_Cherry_MX1A_1.25u_Plate
- SW81: value Left -> KEYSW; footprint Button_Switch_Keyboard:SW_Cherry_MX1A_1.00u_PCB -> Button_Switch_Keyboard:SW_Cherry_MX1A_1.00u_Plate
- SW82: value Down -> KEYSW; footprint Button_Switch_Keyboard:SW_Cherry_MX1A_1.00u_PCB -> Button_Switch_Keyboard:SW_Cherry_MX1A_1.00u_Plate
- SW83: value Right -> KEYSW; footprint Button_Switch_Keyboard:SW_Cherry_MX1A_1.00u_PCB -> Button_Switch_Keyboard:SW_Cherry_MX1A_1.00u_Plate
- SW84: value 0 -> KEYSW; footprint Button_Switch_Keyboard:SW_Cherry_MX1A_2.00u_PCB -> Button_Switch_Keyboard:SW_Cherry_MX1A_2.00u_Plate
- SW85: footprint Button_Switch_Keyboard:SW_Cherry_MX1A_1.00u_PCB -> Button_Switch_Keyboard:SW_Cherry_MX1A_1.00u_Plate
- moved SW_95 406.6 mm to (372.3, 155.6)
- moved R4 394.1 mm to (369.3, 146.1), turned to 270 degrees
- moved R1 387.9 mm to (368.1, 85.5), turned to 270 degrees
- moved J1 387.3 mm to (370.2, 79.2)
- moved R2 386.7 mm to (372.9, 85.5), turned to 270 degrees
- moved C2 100.2 mm to (362.2, 113.4), turned to 90 degrees
- moved C3 97.4 mm to (356.8, 113.4), turned to 90 degrees
- moved C4 97.4 mm to (366.9, 113.4), turned to 270 degrees
- moved C5 84.0 mm to (373.5, 125.9), turned to 0 degrees
- moved MCU1 73.6 mm to (359.9, 126.7), turned to 180 degrees
- moved C1 63.1 mm to (370.7, 138.1), turned to 0 degrees
- moved C7 54.2 mm to (365.3, 139.6), turned to 270 degrees
- moved X1 49.4 mm to (360.3, 139.6), turned to 45 degrees
- moved C6 46.4 mm to (355.3, 139.6)
- moved R3 39.4 mm to (355.7, 146.1), turned to 270 degrees
Connections:
- net Net-(MCU1-Pad17) renamed /MCU/Mosfet
- D56 pad 1: /Keyboard Matrix/row2 -> /Keyboard Matrix/row3
- D57 pad 1: /Keyboard Matrix/row2 -> /Keyboard Matrix/row3
- D58 pad 1: /Keyboard Matrix/row2 -> /Keyboard Matrix/row3
- D59 pad 1: /Keyboard Matrix/row2 -> /Keyboard Matrix/row3
- D60 pad 1: /Keyboard Matrix/row2 -> /Keyboard Matrix/row3
- D61 pad 1: /Keyboard Matrix/row2 -> /Keyboard Matrix/row3
- D62 pad 1: /Keyboard Matrix/row2 -> /Keyboard Matrix/row3
- D63 pad 1: /Keyboard Matrix/row2 -> /Keyboard Matrix/row3
- D64 pad 1: /Keyboard Matrix/row2 -> /Keyboard Matrix/row3
- D65 pad 1: /Keyboard Matrix/row2 -> /Keyboard Matrix/row3
- D66 pad 1: /Keyboard Matrix/row2 -> /Keyboard Matrix/row3
- D67 pad 1: /Keyboard Matrix/row2 -> /Keyboard Matrix/row3
- D68 pad 1: /Keyboard Matrix/row2 -> /Keyboard Matrix/row3
- D69 pad 1: /Keyboard Matrix/row2 -> /Keyboard Matrix/row3
- D70 pad 1: /Keyboard Matrix/row2 -> /Keyboard Matrix/row3
- D71 pad 1: /Keyboard Matrix/row2 -> /Keyboard Matrix/row3
- D72 pad 1: /Keyboard Matrix/row2 -> /Keyboard Matrix/row3
- MCU1 pad 11: Net-(MCU1-Pad11) -> /Keyboard Matrix/col20
- MCU1 pad 12: Net-(MCU1-Pad12) -> /Keyboard Matrix/col19
- MCU1 pad 13: Net-(MCU1-Pad13) -> /Keyboard Matrix/col18
- MCU1 pad 14: Net-(MCU1-Pad14) -> /Keyboard Matrix/col17
- MCU1 pad 15: Net-(MCU1-Pad15) -> /Keyboard Matrix/row3
- MCU1 pad 16: Net-(MCU1-Pad16) -> /Keyboard Matrix/row4
- MCU1 pad 27: /Keyboard Matrix/col20 -> Net-(MCU1-Pad27)
- MCU1 pad 28: /Keyboard Matrix/col19 -> Net-(MCU1-Pad28)
- MCU1 pad 29: /Keyboard Matrix/col18 -> Net-(MCU1-Pad29)
- MCU1 pad 30: /Keyboard Matrix/col17 -> Net-(MCU1-Pad30)
- MCU1 pad 49: Net-(MCU1-Pad49) -> /Keyboard Matrix/row0
- MCU1 pad 50: Net-(MCU1-Pad50) -> /Keyboard Matrix/row1
- MCU1 pad 51: Net-(MCU1-Pad51) -> /Keyboard Matrix/row2
- MCU1 pad 57: /Keyboard Matrix/row4 -> Net-(MCU1-Pad57)
- MCU1 pad 58: /Keyboard Matrix/row2 -> Net-(MCU1-Pad58)
- MCU1 pad 59: /Keyboard Matrix/row2 -> Net-(MCU1-Pad59)
- MCU1 pad 60: /Keyboard Matrix/row1 -> Net-(MCU1-Pad60)
- MCU1 pad 61: /Keyboard Matrix/row0 -> Net-(MCU1-Pad61)
Routing:
- net /Keyboard Matrix/row0: track 0.00 -> 481.9 mm, vias 0 -> 4
- net /Keyboard Matrix/row4: track 0.00 -> 471.1 mm
- net /Keyboard Matrix/row2: track 0.00 -> 450.0 mm, vias 0 -> 3
- net /Keyboard Matrix/row3: track 0.00 -> 441.7 mm, vias 0 -> 2
- net /Keyboard Matrix/row1: track 0.00 -> 435.3 mm, vias 0 -> 4
- net /Keyboard Matrix/col0: track 0.00 -> 428.4 mm
- net /Keyboard Matrix/col1: track 0.00 -> 409.3 mm
- net /Keyboard Matrix/col3: track 0.00 -> 384.0 mm
- net /Keyboard Matrix/col2: track 0.00 -> 378.6 mm
- net /Keyboard Matrix/col4: track 0.00 -> 340.3 mm
- net /Keyboard Matrix/col6: track 0.00 -> 319.5 mm
- net /Keyboard Matrix/col5: track 0.00 -> 318.6 mm
- net /Keyboard Matrix/col7: track 0.00 -> 280.3 mm
- net /Keyboard Matrix/col8: track 0.00 -> 261.3 mm
- net /Keyboard Matrix/col10: track 0.00 -> 197.2 mm
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Other:
- board size 413.2 x 99.8 mm -> 408.5 x 95 mm
- net class Default: trace_width 0.25 -> 0.3
- rule trace_min: 0.2 -> 0.3

Commit message: Leds
Parts:
- added D90: LED, keyboard_parts:SMD_LED_Green_Migist, B.Cu at (83.1, 149.6)
- added D91: LED, keyboard_parts:SMD_LED_Green_Migist, B.Cu at (163.9, 149.6)
- added D92: LED, keyboard_parts:SMD_LED_Green_Migist, B.Cu at (244.6, 149.6)
- added D93: LED, keyboard_parts:SMD_LED_Green_Migist, B.Cu at (327.8, 149.6)
- added D94: LED, keyboard_parts:SMD_LED_Green_Migist, B.Cu at (408.5, 149.6)
- added D95: LED, keyboard_parts:SMD_LED_Green_Migist, B.Cu at (83.1, 92.6)
- added D96: LED, keyboard_parts:SMD_LED_Green_Migist, B.Cu at (163.9, 93.8)
- added D97: LED, keyboard_parts:SMD_LED_Green_Migist, B.Cu at (244.6, 95.0)
- added D98: LED, keyboard_parts:SMD_LED_Green_Migist, B.Cu at (327.8, 95.0)
- added D99: LED, keyboard_parts:SMD_LED_Green_Migist, B.Cu at (408.5, 92.6)
- added Q1: Mosfet, keyboard_parts:MOSFET, B.Cu at (328.0, 123.0)
- added R80: 1k, Resistors_SMD:R_0805_HandSoldering, B.Cu at (337.0, 122.0)
- added R90: R, Resistors_SMD:R_0805_HandSoldering, B.Cu at (91.4, 149.6)
- added R91: R, Resistors_SMD:R_0805_HandSoldering, B.Cu at (172.2, 149.6)
- added R92: R, Resistors_SMD:R_0805_HandSoldering, B.Cu at (252.9, 149.6)
- added R93: R, Resistors_SMD:R_0805_HandSoldering, B.Cu at (336.1, 149.6)
- added R94: R, Resistors_SMD:R_0805_HandSoldering, B.Cu at (416.8, 149.6)
- added R95: R, Resistors_SMD:R_0805_HandSoldering, B.Cu at (91.4, 92.6)
- added R96: R, Resistors_SMD:R_0805_HandSoldering, B.Cu at (171.2, 93.8)
- added R97: R, Resistors_SMD:R_0805_HandSoldering, B.Cu at (257.9, 95.0)
- added R98: R, Resistors_SMD:R_0805_HandSoldering, B.Cu at (336.1, 95.0)
- added R99: R, Resistors_SMD:R_0805_HandSoldering, B.Cu at (416.8, 92.6)
Routing:
- net Net-(D90-Pad1): track 0.00 -> 806.1 mm, vias 0 -> 16
- net VCC: track 115.8 -> 834.1 mm, vias 0 -> 8
- net GND: track 85.2 -> 127.6 mm, vias 6 -> 8
- net /MCU/Mosfet: track 0.00 -> 34.4 mm, vias 0 -> 2
- net Net-(D97-Pad2): track 0.00 -> 10.0 mm
- net Net-(Q1-Pad1): track 0.00 -> 5.72 mm
- net Net-(D95-Pad2): track 0.00 -> 5.09 mm
- net Net-(D92-Pad2): track 0.00 -> 5.09 mm
- net Net-(D91-Pad2): track 0.00 -> 5.09 mm
- net Net-(D90-Pad2): track 0.00 -> 5.09 mm
- net Net-(D99-Pad2): track 0.00 -> 5.09 mm
- net Net-(D98-Pad2): track 0.00 -> 5.09 mm
- net Net-(D94-Pad2): track 0.00 -> 5.09 mm
- net Net-(D93-Pad2): track 0.00 -> 5.09 mm
- net Net-(D96-Pad2): track 0.00 -> 4.06 mm
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
Commit message: 3d Model
Parts:
- added G***: LOGO, keyboard_parts:RG, B.Cu at (280.2, 140.8)
Other:
- board text added: "Migouner 1.0"

Commit message: Keyboard 2
Parts:
- added C8: 0.1u, Capacitors_SMD:C_0805_HandSoldering, B.Cu at (375.4, 126.0)
- moved C5 3.96 mm to (373.4, 121.9), turned to 90 degrees
Connections:
- MCU1 pad 8: Net-(MCU1-Pad8) -> VCC
Routing:
- net VCC: track 834.1 -> 844.5 mm
- net Net-(C5-Pad1): track 4.74 -> 6.73 mm
Other:
- board text added: "Migouner 1.1"
- board text removed: "Migouner 1.0"
