File: keyboard-layout/keyboard-layout-pcb.kicad_pcb (KiCad board)
At the start: 2 copper layers, 408.5 x 95 mm, 211 parts, among them J1 USB_mini_micro_B, Q1 Mosfet, SW0 KEYSW, SW1 KEYSW, SW10 KEYSW, SW11 KEYSW, SW12 KEYSW, SW13 KEYSW, SW14 KEYSW, SW15 KEYSW, SW16 KEYSW, SW17 KEYSW, SW18 KEYSW, SW19 KEYSW, SW2 KEYSW, SW20 KEYSW, SW21 KEYSW, SW22 KEYSW, SW23 KEYSW, SW24 KEYSW, SW25 KEYSW, SW26 KEYSW, SW27 KEYSW, SW28 KEYSW, SW29 KEYSW, SW3 KEYSW, SW30 KEYSW, SW31 KEYSW, SW32 KEYSW, SW33 KEYSW, SW34 KEYSW, SW35 KEYSW, SW36 KEYSW, SW37 KEYSW, SW38 KEYSW, SW39 KEYSW, SW4 KEYSW, SW40 KEYSW, SW41 KEYSW, SW42 KEYSW, SW43 KEYSW, SW44 KEYSW, SW45 KEYSW, SW46 KEYSW, SW47 KEYSW, SW48 KEYSW, SW49 KEYSW, SW5 KEYSW, SW50 KEYSW, SW51 KEYSW, SW52 KEYSW, SW53 KEYSW, SW54 KEYSW, SW55 KEYSW, SW56 KEYSW, SW57 KEYSW, SW58 KEYSW, SW59 KEYSW, SW6 KEYSW, SW60 KEYSW, SW61 KEYSW, SW62 KEYSW, SW63 KEYSW, SW64 KEYSW, SW65 KEYSW, SW66 KEYSW, SW67 KEYSW, SW68 KEYSW, SW69 KEYSW, SW7 KEYSW, SW70 KEYSW, SW71 KEYSW, SW72 KEYSW, SW73 KEYSW, SW74 KEYSW, SW75 KEYSW, SW76 KEYSW, SW77 KEYSW, SW78 KEYSW, SW79 KEYSW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

Commit message: Optimizations
Routing:
- net VCC: track 844.5 -> 942.7 mm, vias 8 -> 12
- net GND: track 127.6 -> 114.5 mm, vias 8 -> 6
Changed lines of the file:
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@@
-(kicad_pcb (version 4) (host pcbnew 4.0.7)
+(kicad_pcb (version 4) (host pcbnew 4.0.7-e2-6376~58~ubuntu16.04.1)
   (general
     (links 336)
     (no_connects 0)
-    (area 40.056249 69.8808 449.175001 168.950001)
+    (area 40.299999 73.549999 448.950001 168.700001)
     (thickness 1.6)
     (drawings 17)
-    (tracks 1013)
+    (tracks 1026)
     (zones 0)
     (modules 211)
@@
     (38 B.Mask user)
     (39 F.Mask user)
-    (40 Dwgs.User user hide)
+    (40 Dwgs.User user)
     (41 Cmts.User user)
     (42 Eco1.User user)
@@
     (pad_to_mask_clearance 0.2)
     (aux_axis_origin 0 0)
+    (grid_origin 367.625519 126.326939)
     (visible_elements FFFFF77F)
     (pcbplotparams
@@
   (gr_line (start 45.125 73.625) (end 444.125 73.625) (angle 90) (layer Edge.Cuts) (width 0.15))
   (gr_line (start 40.375 163.875) (end 40.375 78.375) (angle 90) (layer Edge.Cuts) (width 0.15))
+  (segment (start 369.3125 144.7125) (end 372.988958 144.7125) (width 0.3) (layer B.Cu) (net 1))
+  (segment (start 367.752519 99.529939) (end 366.34375 99.529939) (width 0.3) (layer B.Cu) (net 1))
+  (via (at 367.752519 99.529939) (size 0.6) (drill 0.4) (layers F.Cu B.Cu) (net 1))
+  (segment (start 368.006519 99.529939) (end 367.752519 99.529939) (width 0.3) (layer F.Cu) (net 1))
+  (segment (start 375.753519 107.276939) (end 368.006519 99.529939) (width 0.3) (layer F.Cu) (net 1))
+  (segment (start 375.753519 141.947939) (end 375.753519 107.276939) (width 0.3) (layer F.Cu) (net 1))
+  (segment (start 373.975519 143.725939) (end 375.753519 141.947939) (width 0.3) (layer F.Cu) (net 1))
+  (via (at 373.975519 143.725939) (size 0.6) (drill 0.4) (layers F.Cu B.Cu) (net 1))
+  (segment (start 372.988958 144.7125) (end 373.975519 143.725939) (width 0.3) (layer B.Cu) (net 1))
+  (segment (start 366.34375 99.529939) (end 366.355519 99.529939) (width 0.3) (layer B.Cu) (net 1))
+  (segment (start 366.355519 99.529939) (end 366.34375 99.529939) (width 0.3) (layer B.Cu) (net 1))
+  (segment (start 92.7875 92.625) (end 92.7875 95.164958) (width 0.3) (layer B.Cu) (net 1))
+  (segment (start 95.525519 152.026939) (end 95.525519 152) (width 0.3) (layer B.Cu) (net 1))
+  (segment (start 95.552458 152) (end 95.525519 152.026939) (width 0.3) (layer B.Cu) (net 1))
+  (segment (start 96.252458 152) (end 95.552458 152) (width 0.3) (layer B.Cu) (net 1))
+  (segment (start 98.825519 149.426939) (end 96.252458 152) (width 0.3) (layer B.Cu) (net 1))
+  (via (at 98.825519 149.426939) (size 0.6) (drill 0.4) (layers F.Cu B.Cu) (net 1))
+  (segment (start 98.825519 132.826939) (end 98.825519 149.426939) (width 0.3) (layer F.Cu) (net 1))
+  (segment (start 90.325519 124.326939) (end 98.825519 132.826939) (width 0.3) (layer F.Cu) (net 1))
+  (segment (start 90.325519 105.626939) (end 90.325519 124.326939) (width 0.3) (layer F.Cu) (net 1))
+  (segment (start 90.225519 105.526939) (end 90.325519 105.626939) (width 0.3) (layer F.Cu) (net 1))
+  (via (at 90.225519 105.526939) (size 0.6) (drill 0.4) (layers F.Cu B.Cu) (net 1))
+  (segment (start 90.225519 97.726939) (end 90.225519 105.526939) (width 0.3) (layer B.Cu) (net 1))
+  (segment (start 92.7875 95.164958) (end 90.225519 97.726939) (width 0.3) (layer B.Cu) (net 1))
+  (segment (start 367.625519 126.326939) (end 372.325519 126.326939) (width 0.3) (layer B.Cu) (net 1))
+  (segment (start 372.668458 125.984) (end 374.162 125.984) (width 0.3) (layer B.Cu) (net 1))
+  (segment (start 372.325519 126.326939) (end 372.668458 125.984) (width 0.3) (layer B.Cu) (net 1))
   (segment (start 367.625519 126.326939) (end 364.173061 126.326939) (width 0.3) (layer B.Cu) (net 1))
   (segment (start 364.173061 126.326939) (end 364 126.5) (width 0.3) (layer B.Cu) (net 1))
-  (segment (start 367.625519 126.326939) (end 373.819061 126.326939) (width 0.3) (layer B.Cu) (net 1))
   (segment (start 373.819061 126.326939) (end 374.162 125.984) (width 0.3) (layer B.Cu) (net 1))
   (segment (start 362.687519 134.464939) (end 362.687519 127.812481) (width 0.3) (layer B.Cu) (net 1))
@@
   (segment (start 369.275 144.75) (end 369.3125 144.7125) (width 0.3) (layer B.Cu) (net 1))
   (segment (start 366.9375 152) (end 366.9375 144.75) (width 0.3) (layer B.Cu) (net 1))
-  (segment (start 366.9375 144.75) (end 366.9375 140.614458) (width 0.3) (layer B.Cu) (net 1))
-  (segment (start 366.9375 140.614458) (end 369.450019 138.101939) (width 0.3) (layer B.Cu) (net 1))
   (segment (start 337.4125 95) (end 345.5 95) (width 0.3) (layer B.Cu) (net 1))
   (segment (start 356 94) (end 366.34375 94) (width 0.3) (layer B.Cu) (net 1))
@@
   (segment (start 92.7875 149.625) (end 92.7875 149.4625) (width 0.3) (layer B.Cu) (net 1))
   (segment (start 92.7875 149.4625) (end 95.325 152) (width 0.3) (layer B.Cu) (net 1))
-  (segment (start 95.325 152) (end 171 152) (width 0.3) (layer B.Cu) (net 1))
+  (segment (start 95.325 152) (end 95.525519 152) (width 0.3) (layer B.Cu) (net 1))
+  (segment (start 95.525519 152) (end 171 152) (width 0.3) (layer B.Cu) (net 1))
   (segment (start 171 152) (end 171.1625 152) (width 0.3) (layer B.Cu) (net 1))
   (segment (start 171.1625 152) (end 173.5375 149.625) (width 0.3) (layer B.Cu) (net 1))
   (segment (start 366.9375 112.15625) (end 366.9375 110.4375) (width 0.3) (layer B.Cu) (net 1))
-  (segment (start 366.34375 109.84375) (end 366.34375 94) (width 0.3) (layer B.Cu) (net 1))
   (segment (start 366.9375 110.4375) (end 366.34375 109.84375) (width 0.3) (layer B.Cu) (net 1))
+  (segment (start 366.34375 109.84375) (end 366.34375 99.529939) (width 0.3) (layer B.Cu) (net 1))
+  (segment (start 366.34375 99.529939) (end 366.34375 94) (width 0.3) (layer B.Cu) (net 1))
   (segment (start 366.34375 94) (end 366.34375 81.00625) (width 0.3) (layer B.Cu) (net 1))
   (segment (start 366.34375 81.00625) (end 368.1 79.25) (width 0.3) (layer B.Cu) (net 1))
@@
   (segment (start 356.287519 118.988939) (end 356.287519 120.687519) (width 0.3) (layer B.Cu) (net 1))
   (segment (start 356.287519 120.687519) (end 357.926939 122.326939) (width 0.3) (layer B.Cu) (net 1))
-  (segment (start 362.1875 114.65625) (end 356.84375 114.65625) (width 0.3) (layer B.Cu) (net 1))
   (segment (start 366.9375 112.15625) (end 366.53125 112.15625) (width 0.3) (layer B.Cu) (net 1))
-  (segment (start 366.53125 112.15625) (end 364.03125 114.65625) (width 0.3) (layer B.Cu) (net 1))
-  (segment (start 369.3125 144.7125) (end 369.3125 138.239458) (width 0.3) (layer B.Cu) (net 1))
   (segment (start 369.3125 138.239458) (end 369.450019 138.101939) (width 0.3) (layer B.Cu) (net 1))
   (segment (start 362.687519 134.464939) (end 362.687519 136.468769) (width 0.3) (layer B.Cu) (net 1))
@@
   (segment (start 364.03125 114.65625) (end 362.1875 114.65625) (width 0.3) (layer B.Cu) (net 1))
   (segment (start 365.887519 116.512519) (end 364.03125 114.65625) (width 0.3) (layer B.Cu) (net 1))
-  (segment (start 357.087519 118.988939) (end 357.087519 117.162481) (width 0.3) (layer B.Cu) (net 2))
-  (via (at 359.4 112.2) (size 0.6) (drill 0.4) (layers F.Cu B.Cu) (net 2))
-  (segment (start 359.4 114.85) (end 359.4 112.2) (width 0.3) (layer F.Cu) (net 2))
-  (segment (start 358.75 115.5) (end 359.4 114.85) (width 0.3) (layer F.Cu) (net 2))
-  (via (at 358.75 115.5) (size 0.6) (drill 0.4) (layers F.Cu B.Cu) (net 2))
-  (segment (start 357.087519 117.162481) (end 358.75 115.5) (width 0.3) (layer B.Cu) (net 2))
   (segment (start 371.950019 140.450019) (end 372.25 140.75) (width 0.3) (layer B.Cu) (net 2))
   (via (at 372.25 140.75) (size 0.6) (drill 0.4) (layers F.Cu B.Cu) (net 2))
@@
   (segment (start 368.34375 114.65625) (end 369 114) (width 0.3) (layer B.Cu) (net 2))
   (via (at 369 114) (size 0.6) (drill 0.4) (layers F.Cu B.Cu) (net 2))
-  (segment (start 356.84375 112.15625) (end 359.35625 112.15625) (width 0.3) (layer B.Cu) (net 2))
-  (segment (start 359.35625 112.15625) (end 359.4 112.2) (width 0.3) (layer B.Cu) (net 2))
-  (segment (start 362.1875 112.15625) (end 359.44375 112.15625) (width 0.3) (layer B.Cu) (net 2))
-  (segment (start 359.44375 112.15625) (end 359.4 112.2) (width 0.3) (layer B.Cu) (net 2))
   (segment (start 360.050387 140.945442) (end 360.050387 140.549613) (width 0.3) (layer B.Cu) (net 2))
   (segment (start 360.050387 140.549613) (end 360.2 140.4) (width 0.3) (layer B.Cu) (net 2))
@@
   (segment (start 226.565 99.585) (end 226.565 104.765) (width 0.3) (layer B.Cu) (net 28))
   (segment (start 226.565 104.765) (end 228.675 106.875) (width 0.3) (layer B.Cu) (net 28))
-  (segment (start 375.4 128.2) (end 382.6 128.2) (width 0.3) (layer B.Cu) (net 29))
+  (segment (start 374.991519 128.231939) (end 382.6 128.2) (width 0.3) (layer B.Cu) (net 29))
   (segment (start 355.4 116.4) (end 361.9 116.4) (width 0.3) (layer F.Cu) (net 29))
-  (segment (start 361.9 116.4) (end 373 116.4) (width 0.3) (layer F.Cu) (net 29))
-  (via (at 375.4 128.2) (size 0.6) (drill 0.4) (layers F.Cu B.Cu) (net 29))
-  (segment (start 375.4 118.8) (end 375.4 128.2) (width 0.3) (layer F.Cu) (net 29))
-  (segment (start 373 116.4) (end 375.4 118.8) (width 0.3) (layer F.Cu) (net 29))
+  (segment (start 361.9 116.4) (end 372.197519 116.420939) (width 0.3) (layer F.Cu) (net 29))
+  (via (at 374.991519 128.231939) (size 0.6) (drill 0.4) (layers F.Cu B.Cu) (net 29))
+  (segment (start 374.991519 118.960939) (end 374.991519 128.231939) (width 0.3) (layer F.Cu) (net 29))
+  (segment (start 372.197519 116.420939) (end 374.991519 118.960939) (width 0.3) (layer F.Cu) (net 29))
   (segment (start 355.487519 118.988939) (end 355.487519 116.487519) (width 0.3) (layer B.Cu) (net 29))
   (segment (start 346.375 116.375) (end 315.2 116.375) (width 0.3) (layer B.Cu) (net 29))
