File: keyboard-layout/MCU.sch (KiCad schematic (older format))
At the start: 15 parts, among them J1 USB_mini_micro_B, SW1 SW_PUSH, X1 XTAL_GND

Commit message: Matrix complete
Parts:
- renumbered C3 to C1, C4 to C2, C5 to C3, C6 to C4, C7 to C5, C1 to C6, C2 to C7, R3 to R1, R4 to R2, R2 to R3, R1 to R4
Changed lines of the file:
@@
 LIBS:keyboard_parts
 LIBS:controller-cache
-LIBS:matrix-cache
 EELAYER 25 0
 EELAYER END
@@
 $EndComp
 $Comp
-L C C1
+L C C6
 U 1 1 5B0040BA
 P 5050 6450
-F 0 "C1" H 5075 6550 50  0000 L CNN
+F 0 "C6" H 5075 6550 50  0000 L CNN
 F 1 "22p" H 5075 6350 50  0000 L CNN
 F 2 "Capacitors_SMD:C_0805_HandSoldering" H 5088 6300 50  0001 C CNN
@@
 $EndComp
 $Comp
-L C C2
+L C C7
 U 1 1 5B0040BB
 P 5850 6450
-F 0 "C2" H 5875 6550 50  0000 L CNN
+F 0 "C7" H 5875 6550 50  0000 L CNN
 F 1 "22p" H 5875 6350 50  0000 L CNN
 F 2 "Capacitors_SMD:C_0805_HandSoldering" H 5888 6300 50  0001 C CNN
@@
 $EndComp
 $Comp
-L C C3
+L C C1
 U 1 1 5B0040BD
 P 2350 1550
-F 0 "C3" H 2375 1650 50  0000 L CNN
+F 0 "C1" H 2375 1650 50  0000 L CNN
 F 1 "0.1u" H 2375 1450 50  0000 L CNN
 F 2 "Capacitors_SMD:C_0805_HandSoldering" H 2388 1400 50  0001 C CNN
@@
 $EndComp
 $Comp
-L C C4
+L C C2
 U 1 1 5B0040BE
 P 2650 1550
-F 0 "C4" H 2675 1650 50  0000 L CNN
+F 0 "C2" H 2675 1650 50  0000 L CNN
 F 1 "0.1u" H 2675 1450 50  0000 L CNN
 F 2 "Capacitors_SMD:C_0805_HandSoldering" H 2688 1400 50  0001 C CNN
@@
 $EndComp
 $Comp
-L C C5
+L C C3
 U 1 1 5B0040BF
 P 2950 1550
-F 0 "C5" H 2975 1650 50  0000 L CNN
+F 0 "C3" H 2975 1650 50  0000 L CNN
 F 1 "0.1u" H 2975 1450 50  0000 L CNN
 F 2 "Capacitors_SMD:C_0805_HandSoldering" H 2988 1400 50  0001 C CNN
@@
 $EndComp
 $Comp
-L C C6
+L C C4
 U 1 1 5B0040C0
 P 3250 1550
-F 0 "C6" H 3275 1650 50  0000 L CNN
+F 0 "C4" H 3275 1650 50  0000 L CNN
 F 1 "4.7u" H 3275 1450 50  0000 L CNN
 F 2 "Capacitors_SMD:C_0805_HandSoldering" H 3288 1400 50  0001 C CNN
@@
 $EndComp
 $Comp
-L R R1
+L R R4
 U 1 1 5B0040C4
 P 3400 5750
-F 0 "R1" V 3480 5750 50  0000 C CNN
+F 0 "R4" V 3480 5750 50  0000 C CNN
 F 1 "10k" V 3400 5750 50  0000 C CNN
 F 2 "Resistors_SMD:R_0805_HandSoldering" V 3330 5750 50  0001 C CNN
@@
 $EndComp
 $Comp
-L R R2
+L R R3
 U 1 1 5B0040C7
 P 7050 3450
-F 0 "R2" V 7130 3450 50  0000 C CNN
+F 0 "R3" V 7130 3450 50  0000 C CNN
 F 1 "10k" V 7050 3450 50  0000 C CNN
 F 2 "Resistors_SMD:R_0805_HandSoldering" V 6980 3450 50  0001 C CNN
@@
 $EndComp
 $Comp
-L R R3
+L R R1
 U 1 1 5B0040CB
 P 3050 3150
-F 0 "R3" V 3130 3150 50  0000 C CNN
+F 0 "R1" V 3130 3150 50  0000 C CNN
 F 1 "22" V 3050 3150 50  0000 C CNN
 F 2 "Resistors_SMD:R_0805_HandSoldering" V 2980 3150 50  0001 C CNN
@@
 $EndComp
 $Comp
-L R R4
+L R R2
 U 1 1 5B0040CC
 P 3250 3300
-F 0 "R4" V 3330 3300 50  0000 C CNN
+F 0 "R2" V 3330 3300 50  0000 C CNN
 F 1 "22" V 3250 3300 50  0000 C CNN
 F 2 "Resistors_SMD:R_0805_HandSoldering" V 3180 3300 50  0001 C CNN
@@
 $EndComp
 $Comp
-L C C7
+L C C5
 U 1 1 5B0040CE
 P 3350 3600
-F 0 "C7" H 3375 3700 50  0000 L CNN
+F 0 "C5" H 3375 3700 50  0000 L CNN
 F 1 "1u" H 3375 3500 50  0000 L CNN
 F 2 "Capacitors_SMD:C_0805_HandSoldering" H 3388 3450 50  0001 C CNN

Commit message: pcb progress
Parts:
- X1: footprint Crystals:Crystal_SMD_SeikoEpson_FA238-4pin_3.2x2.5mm -> keyboard_parts:FA-238
- renumbered SW1 to SW_95
Connections:
- net col0: now also MCU1.48 (PA3); no longer MCU1.59 (PF2)
- net col1: now also MCU1.47 (PA4); no longer MCU1.58 (PF3)
- net col20: now reaches MCU1.27 (PD2)
- net col19: now reaches MCU1.28 (PD3)
- net col18: now reaches MCU1.29 (PD4)
- net col17: now reaches MCU1.30 (PD5)
- net col16: now reaches MCU1.31 (PD6)
- net col15: now reaches MCU1.32 (PD7)
- net col14: now reaches MCU1.33 (PE0)
- net col13: now reaches MCU1.34 (PE1)
- net col12: now reaches MCU1.35 (PC0)
- net col11: now reaches MCU1.36 (PC1)
- net col10: now reaches MCU1.37 (PC2)
- net col9: now reaches MCU1.38 (PC3)
- net col8: now reaches MCU1.39 (PC4)
- net col7: now reaches MCU1.40 (PC5)
- net col6: now reaches MCU1.41 (PC6)
- net col5: now reaches MCU1.42 (PC7)
- net col4: now reaches MCU1.44 (PA7)
- net col3: now reaches MCU1.45 (PA6)
- net col2: now reaches MCU1.46 (PA5)
- net row5: now reaches MCU1.56 (PF5)
- net row4: now reaches MCU1.57 (PF4)
- new net row2: MCU1.59 (PF2)
- new net row3: MCU1.58 (PF3)
- no-connect marks 46 -> 23
Changed lines of the file:
@@
 F 0 "X1" H 5450 6450 60  0000 C CNN
 F 1 "XTAL_GND" H 5450 6150 60  0000 C CNN
-F 2 "Crystals:Crystal_SMD_SeikoEpson_FA238-4pin_3.2x2.5mm" H 5450 6300 60  0001 C CNN
+F 2 "keyboard_parts:FA-238" H 5450 6300 60  0001 C CNN
 F 3 "" H 5450 6300 60  0000 C CNN
 	1    5450 6300
@@
 $EndComp
 $Comp
-L SW_PUSH SW1
+L SW_PUSH SW_95
 U 1 1 5B0040C3
 P 3400 6050
-F 0 "SW1" H 3550 6160 50  0000 C CNN
+F 0 "SW_95" H 3550 6160 50  0000 C CNN
 F 1 "SW_PUSH" H 3400 5970 50  0000 C CNN
 F 2 "Buttons_Switches_SMD:SW_SPST_TL3342" H 3400 6050 60  0001 C CNN
@@
 	0    -1   -1   0
 $EndComp
-Text Notes 6800 3300 0    60   ~ 0
+Text Notes 7650 3500 0    60   ~ 0
 HWB (Bootloader)
 $Comp
@@
 $EndComp
 NoConn ~ 4300 2200
-NoConn ~ 5050 2200
-NoConn ~ 5200 2200
-NoConn ~ 5350 2200
 NoConn ~ 5500 2200
 NoConn ~ 5950 2200
 NoConn ~ 6100 2200
 NoConn ~ 6250 2200
-NoConn ~ 6600 2700
-NoConn ~ 6600 2850
-NoConn ~ 6600 3000
-NoConn ~ 6600 3150
-NoConn ~ 6600 3300
-NoConn ~ 6600 3600
-NoConn ~ 6600 3750
-NoConn ~ 6600 3900
-NoConn ~ 6600 4050
-NoConn ~ 6600 4200
-NoConn ~ 6600 4350
-NoConn ~ 6600 4500
-NoConn ~ 6600 4650
-NoConn ~ 6600 4800
-NoConn ~ 6600 4950
-NoConn ~ 6250 5450
-NoConn ~ 6100 5450
-NoConn ~ 5950 5450
-NoConn ~ 5800 5450
-NoConn ~ 5650 5450
-NoConn ~ 5500 5450
 NoConn ~ 5350 5450
 NoConn ~ 5200 5450
@@
 Text HLabel 4600 1900 1    60   Input ~ 0
 row1
-Text HLabel 4750 1900 1    60   Input ~ 0
-col0
-Text HLabel 4900 1900 1    60   Input ~ 0
-col1
-Wire Wire Line
-	4900 2200 4900 1900
-Wire Wire Line
-	4750 2200 4750 1900
 Wire Wire Line
 	4600 2200 4600 1900
@@
 	5050 6300 5150 6300
 NoConn ~ 2500 3350
+Text HLabel 4750 1900 1    60   Input ~ 0
+row2
+Text HLabel 4900 1900 1    60   Input ~ 0
+row3
+Text HLabel 5050 1900 1    60   Input ~ 0
+row4
+Text HLabel 5200 1900 1    60   Input ~ 0
+row5
+Wire Wire Line
+	4750 1900 4750 2200
+Wire Wire Line
+	4900 1900 4900 2200
+Wire Wire Line
+	5050 2200 5050 1900
+Wire Wire Line
+	5200 1900 5200 2200
+NoConn ~ 5350 2200
+Text HLabel 6850 2700 2    60   Input ~ 0
+col0
+Text HLabel 6850 2850 2    60   Input ~ 0
+col1
+Text HLabel 6850 3000 2    60   Input ~ 0
+col2
+Text HLabel 6850 3150 2    60   Input ~ 0
+col3
+Text HLabel 6850 3300 2    60   Input ~ 0
+col4
+Text HLabel 6850 3600 2    60   Input ~ 0
+col5
+Text HLabel 6850 3750 2    60   Input ~ 0
+col6
+Text HLabel 6850 3900 2    60   Input ~ 0
+col7
+Text HLabel 6850 4050 2    60   Input ~ 0
+col8
+Text HLabel 6850 4200 2    60   Input ~ 0
+col9
+Text HLabel 6850 4350 2    60   Input ~ 0
+col10
+Text HLabel 6850 4500 2    60   Input ~ 0
+col11
+Text HLabel 6850 4650 2    60   Input ~ 0
+col12
+Text HLabel 6850 4800 2    60   Input ~ 0
+col13
+Text HLabel 6850 4950 2    60   Input ~ 0
+col14
+Text HLabel 6250 5700 3    60   Input ~ 0
+col15
+Text HLabel 6100 5700 3    60   Input ~ 0
+col16
+Text HLabel 5950 5700 3    60   Input ~ 0
+col17
+Text HLabel 5800 5700 3    60   Input ~ 0
+col18
+Text HLabel 5650 5700 3    60   Input ~ 0
+col19
+Text HLabel 5500 5700 3    60   Input ~ 0
+col20
+Wire Wire Line
+	6600 2700 6850 2700
+Wire Wire Line
+	6600 2850 6850 2850
+Wire Wire Line
+	6600 3000 6850 3000
+Wire Wire Line
+	6600 3150 6850 3150
+Wire Wire Line
+	6600 3300 6850 3300
+Wire Wire Line
+	6600 3600 6850 3600
+Wire Wire Line
+	6850 3750 6600 3750
+Wire Wire Line
+	6600 3900 6850 3900
+Wire Wire Line
+	6600 4050 6850 4050
+Wire Wire Line
+	6600 4200 6850 4200
+Wire Wire Line
+	6600 4350 6850 4350
+Wire Wire Line
+	6850 4500 6600 4500
+Wire Wire Line
+	6600 4650 6850 4650
+Wire Wire Line
+	6850 4800 6600 4800
+Wire Wire Line
+	6600 4950 6850 4950
+Wire Wire Line
+	6250 5700 6250 5450
+Wire Wire Line
+	6100 5450 6100 5700
+Wire Wire Line
+	5950 5450 5950 5700
+Wire Wire Line
+	5800 5450 5800 5700
+Wire Wire Line
+	5650 5700 5650 5450
+Wire Wire Line
+	5500 5450 5500 5700
 $EndSCHEMATC

Commit message: python scripting
Connections:
- net row5: no longer names the net of MCU1.56 (PF5)
- no-connect marks 23 -> 24
Changed lines of the file:
@@
 Text HLabel 5050 1900 1    60   Input ~ 0
 row4
-Text HLabel 5200 1900 1    60   Input ~ 0
-row5
 Wire Wire Line
 	4750 1900 4750 2200
@@
 Wire Wire Line
 	5050 2200 5050 1900
-Wire Wire Line
-	5200 1900 5200 2200
 NoConn ~ 5350 2200
 Text HLabel 6850 2700 2    60   Input ~ 0
@@
 Wire Wire Line
 	5500 5450 5500 5700
+NoConn ~ 5200 2200
 $EndSCHEMATC

Commit message: pcb without leds finished
Connections:
- net col17: now also MCU1.14 (PB4); no longer MCU1.30 (PD5)
- net col18: now also MCU1.13 (PB3); no longer MCU1.29 (PD4)
- net col19: now also MCU1.12 (PB2); no longer MCU1.28 (PD3)
- net col20: now also MCU1.11 (PB1); no longer MCU1.27 (PD2)
- net row0: now also MCU1.49 (PA2); no longer MCU1.61 (PF0)
- net row1: now also MCU1.50 (PA1); no longer MCU1.60 (PF1)
- net row2: now also MCU1.51 (PA0); no longer MCU1.59 (PF2)
- net row3: now also MCU1.15 (PB5); no longer MCU1.58 (PF3)
- net row4: now also MCU1.16 (PB6); no longer MCU1.57 (PF4)
- net Mosfet: now reaches MCU1.17 (PB7)
- no-connect marks 24 -> 23
Changed lines of the file:
@@
 $Descr A4 11693 8268
 encoding utf-8
-Sheet 3 3
+Sheet 2 3
 Title ""
 Date ""
@@
 NoConn ~ 4300 2200
 NoConn ~ 5500 2200
-NoConn ~ 5950 2200
-NoConn ~ 6100 2200
-NoConn ~ 6250 2200
+NoConn ~ 4450 2200
+NoConn ~ 4600 2200
+NoConn ~ 4750 2200
 NoConn ~ 5350 5450
 NoConn ~ 5200 5450
-NoConn ~ 4300 5450
-NoConn ~ 4150 5450
-NoConn ~ 4000 5450
-NoConn ~ 3650 4950
-NoConn ~ 3650 4800
-NoConn ~ 3650 4650
-NoConn ~ 3650 4500
-NoConn ~ 3650 4350
-NoConn ~ 3650 4200
+NoConn ~ 5050 2200
+NoConn ~ 4900 2200
 NoConn ~ 3650 4050
 NoConn ~ 3650 3900
@@
 NoConn ~ 3650 2850
 NoConn ~ 3650 2700
-Text HLabel 4450 1900 1    60   Input ~ 0
+Text HLabel 6250 2200 1    60   Input ~ 0
 row0
-Text HLabel 4600 1900 1    60   Input ~ 0
+Text HLabel 6100 2200 1    60   Input ~ 0
 row1
-Wire Wire Line
-	4600 2200 4600 1900
-Wire Wire Line
-	4450 2200 4450 1900
 Wire Wire Line
 	5650 2200 5650 1800
@@
 	5050 6300 5150 6300
 NoConn ~ 2500 3350
-Text HLabel 4750 1900 1    60   Input ~ 0
-row2
-Text HLabel 4900 1900 1    60   Input ~ 0
-row3
-Text HLabel 5050 1900 1    60   Input ~ 0
-row4
-Wire Wire Line
-	4750 1900 4750 2200
-Wire Wire Line
-	4900 1900 4900 2200
-Wire Wire Line
-	5050 2200 5050 1900
 NoConn ~ 5350 2200
 Text HLabel 6850 2700 2    60   Input ~ 0
@@
 Text HLabel 6100 5700 3    60   Input ~ 0
 col16
-Text HLabel 5950 5700 3    60   Input ~ 0
+Text HLabel 3650 4650 0    60   Input ~ 0
 col17
-Text HLabel 5800 5700 3    60   Input ~ 0
+Text HLabel 3650 4500 0    60   Input ~ 0
 col18
-Text HLabel 5650 5700 3    60   Input ~ 0
+Text HLabel 3650 4350 0    60   Input ~ 0
 col19
-Text HLabel 5500 5700 3    60   Input ~ 0
+Text HLabel 3650 4200 0    60   Input ~ 0
 col20
 Wire Wire Line
@@
 Wire Wire Line
 	6100 5450 6100 5700
-Wire Wire Line
-	5950 5450 5950 5700
-Wire Wire Line
-	5800 5450 5800 5700
-Wire Wire Line
-	5650 5700 5650 5450
-Wire Wire Line
-	5500 5450 5500 5700
 NoConn ~ 5200 2200
+Text HLabel 5950 2200 1    60   Input ~ 0
+row2
+Text HLabel 3650 4800 0    60   Input ~ 0
+row3
+Text HLabel 3650 4950 0    60   Input ~ 0
+row4
+Text HLabel 4000 5450 3    60   Input ~ 0
+Mosfet
+NoConn ~ 5500 5450
+NoConn ~ 5650 5450
+NoConn ~ 5800 5450
+NoConn ~ 5950 5450
+NoConn ~ 4300 5450
+NoConn ~ 4150 5450
 $EndSCHEMATC

Commit message: Keyboard 2
Parts:
- added C8: 0.1u, Capacitors_SMD:C_0805_HandSoldering, symbol C
Connections:
- net GND: now also C8.2
- net VCC: now also MCU1.8 (VBus), C8.1
- no-connect marks 23 -> 22
Other:
- moved on the sheet: C4
Changed lines of the file:
@@
 L C C4
 U 1 1 5B0040C0
-P 3250 1550
-F 0 "C4" H 3275 1650 50  0000 L CNN
-F 1 "4.7u" H 3275 1450 50  0000 L CNN
-F 2 "Capacitors_SMD:C_0805_HandSoldering" H 3288 1400 50  0001 C CNN
-F 3 "" H 3250 1550 50  0001 C CNN
-	1    3250 1550
+P 3550 1550
+F 0 "C4" H 3575 1650 50  0000 L CNN
+F 1 "4.7u" H 3575 1450 50  0000 L CNN
+F 2 "Capacitors_SMD:C_0805_HandSoldering" H 3588 1400 50  0001 C CNN
+F 3 "" H 3550 1550 50  0001 C CNN
+	1    3550 1550
 	1    0    0    -1
 $EndComp
@@
 NoConn ~ 3650 4050
 NoConn ~ 3650 3900
-NoConn ~ 3650 3750
 NoConn ~ 3650 2850
 NoConn ~ 3650 2700
@@
 	2350 1700 2350 1850
 Wire Wire Line
-	2350 1750 3250 1750
+	2350 1750 3550 1750
 Wire Wire Line
 	3250 1750 3250 1700
@@
 Connection ~ 2350 1350
 Wire Wire Line
-	2350 1350 3250 1350
+	2350 1350 3550 1350
 Wire Wire Line
 	2350 1250 2350 1400
@@
 NoConn ~ 4300 5450
 NoConn ~ 4150 5450
+$Comp
+L C C8
+U 1 1 5B746F42
+P 3250 1550
+F 0 "C8" H 3275 1650 50  0000 L CNN
+F 1 "0.1u" H 3275 1450 50  0000 L CNN
+F 2 "Capacitors_SMD:C_0805_HandSoldering" H 3288 1400 50  0001 C CNN
+F 3 "" H 3250 1550 50  0001 C CNN
+	1    3250 1550
+	1    0    0    -1
+$EndComp
+Wire Wire Line
+	3550 1350 3550 1400
+Connection ~ 3250 1350
+Wire Wire Line
+	3550 1750 3550 1700
+Connection ~ 3250 1750
+$Comp
+L VCC #PWR?
+U 1 1 5B747708
+P 3050 3750
+F 0 "#PWR?" H 3050 3600 50  0001 C CNN
+F 1 "VCC" H 3050 3900 50  0000 C CNN
+F 2 "" H 3050 3750 50  0001 C CNN
+F 3 "" H 3050 3750 50  0001 C CNN
+	1    3050 3750
+	0    -1   -1   0
+$EndComp
+Wire Wire Line
+	3650 3750 3050 3750
 $EndSCHEMATC
